File: handmade01/main.kicad_pcb (KiCad board)
At the start: 2 copper layers, 64.8 x 70.1 mm, 69 parts, among them CON1 MicroSD, CON2 MicroSD, J1 JACK_TRS_6PINS, P1 VOLUMN, P4 USB_OTG, P6 UART_DEBUG, Q1 1AM, SW1 Power, SW10 R, SW11 A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

Commit message: 20171208
Parts:
- P4: footprint MyFT_MiniUSB_B -> MyFT_USB_Micro-B
- moved P4 1.30 mm to (150.6, 71.6), turned to 180 degrees
Changed lines of the file:
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@@
-    )
-  )
-  (module MyFT_MiniUSB_B (layer F.Cu)
-    (at 149.352 71.882 90)
-    (descr "USB Mini-B 5-pin SMD connector")
-    (tags "USB USB_B USB_Mini connector")
-    (attr smd)
-    (fp_text reference P4 (at -0.65 6.9 90) (layer F.SilkS)
-      (effects (font (size 1 1) (thickness 0.15)))
-    )
-    (fp_text value USB_OTG (at -0.65 -7.1 90) (layer F.SilkS)
-      (effects (font (size 1 1) (thickness 0.15)))
-    )
-    (fp_line (start -5.5 -5.7) (end 4.2 -5.7) (layer F.SilkS) (width 0.05))
-    (fp_line (start 4.2 -5.7) (end 4.2 5.7) (layer F.SilkS) (width 0.05))
-    (fp_line (start 4.2 5.7) (end -5.5 5.7) (layer F.SilkS) (width 0.05))
-    (fp_line (start -5.5 5.7) (end -5.5 -5.7) (layer F.SilkS) (width 0.05))
-    (fp_line (start -4.25 -3.85) (end -4.25 3.85) (layer F.SilkS) (width 0.12))
-    (fp_line (start -5.25 -3.85) (end -5.25 3.85) (layer F.SilkS) (width 0.12))
-    (fp_line (start -5.25 3.85) (end 3.95 3.85) (layer F.SilkS) (width 0.12))
-    (fp_line (start 3.95 3.85) (end 3.95 -3.85) (layer F.SilkS) (width 0.12))
-    (fp_line (start 3.95 -3.85) (end -5.25 -3.85) (layer F.SilkS) (width 0.12))
-    (pad 1 smd rect (at 2.8 -1.6 90) (size 2.3 0.5)
-      (layers F.Cu F.Paste F.Mask)
-      (net 2 +5V)
-    )
-    (pad 2 smd rect (at 2.8 -0.8 90) (size 2.3 0.5)
-      (layers F.Cu F.Paste F.Mask)
-      (net 84 USB_DM)
-    )
-    (pad 3 smd rect (at 2.8 0 90) (size 2.3 0.5)
-      (layers F.Cu F.Paste F.Mask)
-      (net 85 USB_DP)
-    )
-    (pad 4 smd rect (at 2.8 0.8 90) (size 2.3 0.5)
-      (layers F.Cu F.Paste F.Mask)
-      (net 12 GND)
-    )
-    (pad 5 smd rect (at 2.8 1.6 90) (size 2.3 0.5)
-      (layers F.Cu F.Paste F.Mask)
-      (net 12 GND)
-    )
-    (pad 6 smd rect (at 2.7 -4.45 90) (size 2.5 2)
-      (layers F.Cu F.Paste F.Mask)
-      (net 12 GND)
-    )
-    (pad 6 smd rect (at -2.8 -4.45 90) (size 2.5 2)
-      (layers F.Cu F.Paste F.Mask)
-      (net 12 GND)
-    )
-    (pad 6 smd rect (at 2.7 4.45 90) (size 2.5 2)
-      (layers F.Cu F.Paste F.Mask)
-      (net 12 GND)
-    )
-    (pad 6 smd rect (at -2.8 4.45 90) (size 2.5 2)
-      (layers F.Cu F.Paste F.Mask)
-      (net 12 GND)
     )
   )
@@
     )
   )
+  (module MyFT_USB_Micro-B (layer F.Cu)
+    (at 150.622 71.628 180)
+    (descr "Micro USB Type B Receptacle")
+    (tags "USB USB_B USB_micro USB_OTG")
+    (attr smd)
+    (fp_text reference P4 (at 0 -3.45 180) (layer F.SilkS)
+      (effects (font (size 1 1) (thickness 0.15)))
+    )
+    (fp_text value USB_OTG (at 0 4.8 180) (layer F.SilkS)
+      (effects (font (size 1 1) (thickness 0.15)))
+    )
+    (fp_line (start -4.6 -2.8) (end 4.6 -2.8) (layer F.SilkS) (width 0.05))
+    (fp_line (start 4.6 -2.8) (end 4.6 4.05) (layer F.SilkS) (width 0.05))
+    (fp_line (start 4.6 4.05) (end -4.6 4.05) (layer F.SilkS) (width 0.05))
+    (fp_line (start -4.6 4.05) (end -4.6 -2.8) (layer F.SilkS) (width 0.05))
+    (fp_line (start -4.3509 3.81746) (end 4.3491 3.81746) (layer F.SilkS) (width 0.15))
+    (fp_line (start -4.3509 -2.58754) (end 4.3491 -2.58754) (layer F.SilkS) (width 0.15))
+    (fp_line (start 4.3491 -2.58754) (end 4.3491 3.81746) (layer F.SilkS) (width 0.15))
+    (fp_line (start 4.3491 2.58746) (end -4.3509 2.58746) (layer F.SilkS) (width 0.15))
+    (fp_line (start -4.3509 3.81746) (end -4.3509 -2.58754) (layer F.SilkS) (width 0.15))
+    (pad 1 smd rect (at -1.3009 -1.56254 270) (size 1.35 0.4)
+      (layers F.Cu F.Paste F.Mask)
+      (net 2 +5V)
+    )
+    (pad 2 smd rect (at -0.6509 -1.56254 270) (size 1.35 0.4)
+      (layers F.Cu F.Paste F.Mask)
+      (net 84 USB_DM)
+    )
+    (pad 3 smd rect (at -0.0009 -1.56254 270) (size 1.35 0.4)
+      (layers F.Cu F.Paste F.Mask)
+      (net 85 USB_DP)
+    )
+    (pad 4 smd rect (at 0.6491 -1.56254 270) (size 1.35 0.4)
+      (layers F.Cu F.Paste F.Mask)
+      (net 12 GND)
+    )
+    (pad 5 smd rect (at 1.2991 -1.56254 270) (size 1.35 0.4)
+      (layers F.Cu F.Paste F.Mask)
+      (net 12 GND)
+    )
+    (pad 6 thru_hole oval (at -2.5009 -1.56254 270) (size 0.95 1.25) (drill oval 0.55 0.85)
+      (layers *.Cu *.Mask)
+      (net 12 GND)
+    )
+    (pad 6 thru_hole oval (at 2.4991 -1.56254 270) (size 0.95 1.25) (drill oval 0.55 0.85)
+      (layers *.Cu *.Mask)
+      (net 12 GND)
+    )
+    (pad 6 thru_hole oval (at -3.5009 1.13746 270) (size 1.55 1) (drill oval 1.15 0.5)
+      (layers *.Cu *.Mask)
+      (net 12 GND)
+    )
+    (pad 6 thru_hole oval (at 3.4991 1.13746 270) (size 1.55 1) (drill oval 1.15 0.5)
+      (layers *.Cu *.Mask)
+      (net 12 GND)
+    )
+  )

Commit message: 20090101
Parts:
- moved R15 5.48 mm to (187.2, 84.1)
Changed lines of the file:
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@@
     (pad_to_mask_clearance 0)
     (aux_axis_origin 0 0)
-    (visible_elements FFFFFBBF)
+    (visible_elements 7FFFFFFF)
     (pcbplotparams
       (layerselection 3178497)
@@
   )
   (module MyFT_R_0603 (layer F.Cu)
-    (at 182.626 87.122)
+    (at 187.198 84.0994)
     (descr "C 0603 Hand Soldering")
     (tags 0603)

Commit message: 20171211
Parts:
- R11, R15, R17, R19, R21, R23, R25, R5, R6, R7, R8, R9: moved to B.Cu
- moved R15 91.6 mm to (111.5, 135.6), turned to 270 degrees
- moved C5 91.5 mm to (111.8, 88.6), turned to 90 degrees
- moved R19 80.6 mm to (115.1, 135.6), turned to 270 degrees
- moved P6 76.7 mm to (143.0, 68.8)
- moved C1 72.1 mm to (171.4, 102.4)
- moved C7 71.5 mm to (174.2, 107.7), turned to 270 degrees
- moved R22 70.6 mm to (118.9, 75.4), turned to 90 degrees
- moved R20 67.7 mm to (174.0, 75.4), turned to 90 degrees
- moved R26 67.3 mm to (129.5, 126.2), turned to 270 degrees
- moved R21 66.8 mm to (116.8, 135.6), turned to 270 degrees
- moved R4 64.3 mm to (142.0, 73.2), turned to 90 degrees
- moved C11 57.6 mm to (153.9, 78.0), turned to 180 degrees
- moved C10 56.7 mm to (163.1, 114.0), turned to 90 degrees
- moved R25 56.7 mm to (120.4, 135.6), turned to 270 degrees
- moved U1 52.1 mm to (167.6, 108.0), turned to 180 degrees
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
Commit message: 20171211
Parts:
- moved C8 0.25 mm to (174.2, 103.6)
- moved R2 0.25 mm to (172.7, 105.2)

Commit message: 20171212
Other:
- board text added: "Handmade01 Steward 20171212"
Changed lines of the file:
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@@
     (area 109.9595 65.594999 175.842001 141.073626)
     (thickness 1.6)
-    (drawings 14)
+    (drawings 15)
     (tracks 0)
     (zones 0)
@@
     (pad_to_mask_clearance 0)
     (aux_axis_origin 0 0)
-    (visible_elements 7FFFFBFF)
+    (visible_elements 7FFFFFFF)
     (pcbplotparams
-      (layerselection 3178497)
-      (usegerberextensions true)
+      (layerselection 536838145)
+      (usegerberextensions false)
       (excludeedgelayer true)
       (linewidth 0.100000)
@@
       (padsonsilk false)
       (subtractmaskfromsilk false)
-      (outputformat 1)
+      (outputformat 5)
       (mirror false)
-      (drillshape 1)
+      (drillshape 2)
       (scaleselection 1)
       (outputdirectory ""))
@@
     )
   )
+  (gr_text "Handmade01\nSteward 20171212" (at 143.256 93.726) (layer Dwgs.User)
+    (effects (font (size 1.5 1.5) (thickness 0.3)))
+  )
   (gr_circle (center 116.84 115.062) (end 120.396 115.57) (layer Edge.Cuts) (width 0.1))

Commit message: 20171213
Parts:
- moved R15 1.78 mm to (113.3, 135.6), turned to 90 degrees
- moved R17 1.78 mm to (111.5, 135.6), turned to 90 degrees
- moved R19 1.78 mm to (116.8, 135.6), turned to 90 degrees
- moved R21 1.78 mm to (115.1, 135.6), turned to 90 degrees
- moved R23 1.78 mm to (120.4, 135.6), turned to 90 degrees
- moved R25 1.78 mm to (118.6, 135.6), turned to 90 degrees
- moved R11 1.78 mm to (172.5, 135.6), turned to 90 degrees
- moved R5 1.78 mm to (167.1, 135.6), turned to 90 degrees
- moved R6 1.78 mm to (165.4, 135.6), turned to 90 degrees
- moved R7 1.78 mm to (170.7, 135.6), turned to 90 degrees
- moved R8 1.78 mm to (168.9, 135.6), turned to 90 degrees
- moved R9 1.52 mm to (174.0, 135.6), turned to 90 degrees
- turned R3 to 270 degrees
Routing:
- net SD0_CMD: track 0.00 -> 17.6 mm, vias 0 -> 1
- net SD0_DAT1: track 0.00 -> 17.1 mm, vias 0 -> 1
- net SD0_CLK: track 0.00 -> 17.0 mm, vias 0 -> 1
- net SD0_DAT3: track 0.00 -> 16.9 mm, vias 0 -> 1
- net SD0_DAT0: track 0.00 -> 16.7 mm, vias 0 -> 1
- net SD0_DAT2: track 0.00 -> 16.3 mm, vias 0 -> 1
- net GND: track 0.00 -> 15.9 mm
- net SD1_CMD: track 0.00 -> 14.1 mm, vias 0 -> 1
- net SD1_DAT2: track 0.00 -> 13.4 mm, vias 0 -> 1
- net SD1_DAT3: track 0.00 -> 12.8 mm, vias 0 -> 1
- net SD1_CLK: track 0.00 -> 12.7 mm, vias 0 -> 1
- net SD1_DAT1: track 0.00 -> 12.4 mm, vias 0 -> 1
- net SD1_DAT0: track 0.00 -> 12.2 mm, vias 0 -> 1
- net RTC_+: track 0.00 -> 4.89 mm
- net MUTE: track 0.00 -> 3.82 mm
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Other:
- net class Default: clearance 0.254 -> 0.2; trace_width 0.254 -> 0.2; via_dia 0.889 -> 0.5; via_drill 0.635 -> 0.3
- rule trace_clearance: 0.254 -> 0.2
- rule trace_min: 0.254 -> 0.2
- rule via_min_drill: 0.508 -> 0.3
- rule via_min_size: 0.889 -> 0.5

Commit message: 20090101
Parts:
- moved R24 2.22 mm to (124.1, 120.5)
Routing:
- net SD1_DAT1: track 12.4 -> 19.4 mm
- net SD0_CLK: track 17.0 -> 23.2 mm
- net SD0_DAT3: track 16.9 -> 22.6 mm
- net SD1_CMD: track 14.1 -> 19.3 mm
- net SD0_CMD: track 17.6 -> 21.4 mm
- net SD0_DAT2: track 16.3 -> 19.9 mm
- net SD1_DAT0: track 12.2 -> 14.8 mm
- net N-000001: track 0.00 -> 1.95 mm
- net SD1_DAT3: track 12.8 -> 14.4 mm
- net SD0_DAT0: track 16.7 -> 18.1 mm
- net SD1_DAT2: track 13.4 -> 14.4 mm
