File: handmade01/main.kicad_pcb (KiCad board)
At the start: 2 copper layers, 48 parts, among them CON1 MicroSD, CON2 MicroSD, J1 JACK_TRS_6PINS, P1 VOLUMN, P4 USB_OTG, P6 UART_DEBUG, Q1 1AM, SW1 POWER, SW10 R, SW11 A, SW12 B, SW13 X, SW14 Y, SW2 RESET, SW3 UP, SW4 DOWN, SW5 LEFT, SW6 RIGHT, SW7 SELECT, SW8 START, SW9 L, U1 PCM5102A, U2 PAM8403, U3 IPS_2.4_240x320_ST7789V, U4 CM3354, U5 TPS71718

Commit message: 20171129
Parts:
- removed RN1: SD0_4.7K, Connectors_Molex:Molex_KK-6410-07_07x2.54mm_Straight
- removed RN2: SD1_4.7K, Connectors_Molex:Molex_KK-6410-07_07x2.54mm_Straight
- removed RN3: GAMEPAD_4.7K, Connectors_Molex:Molex_KK-6410-13_13x2.54mm_Straight
- added R10, R11, R12, R13, R14, R15, R16, R17, R18, R19, R20, R21, R22, R23, R24, R25, R26, R27, R28, R5, R6, R7, R8, R9: 4.7K, Resistors_SMD:R_0603_HandSoldering, F.Cu at (149.2, 147.2)
- moved C1 118.4 mm to (233.7, 85.1)
- moved C10 118.4 mm to (219.7, 118.1)
- moved C12 118.4 mm to (223.5, 82.5)
- moved C9 118.4 mm to (219.7, 102.9)
- moved R1 118.4 mm to (209.6, 96.5)
- moved C11 118.4 mm to (218.4, 125.7)
- moved C4 118.4 mm to (212.1, 109.2)
- moved C5 118.4 mm to (229.9, 141.0)
- moved C6 118.4 mm to (212.1, 121.9)
- moved C8 118.4 mm to (218.4, 110.5)
- moved R2 118.4 mm to (240.0, 83.8)
- moved SW11 118.4 mm to (196.8, 135.9)
- moved SW14 118.4 mm to (214.6, 144.8)
- moved SW5 118.4 mm to (232.4, 76.2)
- moved SW6 118.4 mm to (200.7, 125.7)
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Other:
- board outline added: 64.8 x 69.8 mm
- board text added: "20171129"
- board text added: "Handmade01"

Commit message: 20171130
Parts:
- CON1, CON2: footprint Connectors:microSD_Card_Receptacle_Wuerth_693072010801 -> mylib:microsd
- SW1, SW10, SW9: footprint Buttons_Switches_THT:SW_Tactile_SKHH_Angled -> Buttons_Switches_THT:SW_PUSH_6mm
- SW11, SW12, SW3: moved to B.Cu
- SW13: footprint mylib:dpad-v -> mylib:dpad-h; moved to B.Cu
- SW14: footprint mylib:dpad-h -> mylib:dpad-v; moved to B.Cu
- SW2: value RESET -> Reset; footprint Buttons_Switches_THT:SW_Tactile_SPST_Angled_PTS645Vx31-2LFS -> Buttons_Switches_THT:SW_PUSH_6mm
- SW4: value DOWN -> Down; moved to B.Cu
- SW5: value LEFT -> Left; moved to B.Cu
- SW6: value RIGHT -> Right; moved to B.Cu
- SW7: value SELECT -> Select; footprint Buttons_Switches_SMD:SW_SPST_SKQG -> Buttons_Switches_SMD:SW_SPST_TL3342; moved to B.Cu
- SW8: value START -> Start; footprint Buttons_Switches_SMD:SW_SPST_SKQG -> Buttons_Switches_SMD:SW_SPST_TL3342; moved to B.Cu
- U5: footprint Housings_SOIC:SO-5_4.4x3.6mm_Pitch1.27mm -> mylib:sc-70-5
- moved SW5 92.5 mm to (167.6, 142.2)
- moved C5 80.5 mm to (149.9, 132.1)
- moved SW14 60.0 mm to (154.9, 151.1)
- moved SW9 58.5 mm to (105.4, 95.2)
- moved C11 56.7 mm to (186.7, 78.7)
- moved R2 54.3 mm to (188.0, 99.1)
- moved SW8 47.1 mm to (105.4, 129.5)
- moved SW6 46.9 mm to (161.3, 151.1)
- moved C8 44.4 mm to (191.8, 74.9)
- moved R21 44.3 mm to (105.4, 153.7)
- moved R28 43.9 mm to (105.4, 149.9)
- moved R6 43.8 mm to (105.4, 146.1)
- moved C4 42.7 mm to (186.7, 74.9)
- moved C1 42.4 mm to (191.8, 78.7)
- moved SW11 42.4 mm to (154.9, 142.2)
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Connections:
- SW1 pad 1: (no net) -> POWER
- SW1 pad 2: (no net) -> GND
- SW10 pad 1: (no net) -> R
- SW10 pad 2: (no net) -> GND
- SW11 pad 1: (no net) -> A
- SW11 pad 2: (no net) -> GND
- SW12 pad 1: (no net) -> B
- SW12 pad 2: (no net) -> GND
- SW13 pad 1: (no net) -> X
- SW13 pad 2: (no net) -> GND
- SW14 pad 1: (no net) -> Y
- SW14 pad 2: (no net) -> GND
- SW2 pad 1: (no net) -> RESET
- SW2 pad 2: (no net) -> GND
- SW3 pad 1: (no net) -> UP
- SW3 pad 2: (no net) -> GND
- SW5 pad 1: (no net) -> LEFT
- SW5 pad 2: (no net) -> GND
- SW6 pad 1: (no net) -> RIGHT
- SW6 pad 2: (no net) -> GND
- SW7 pad 1: (no net) -> SELECT
- SW7 pad 2: (no net) -> GND
- SW8 pad 1: (no net) -> START
- SW8 pad 2: (no net) -> GND
- SW9 pad 1: (no net) -> L
- SW9 pad 2: (no net) -> GND
- U4 pad 11: (no net) -> POWER
- U4 pad 48: (no net) -> SD0_CD
- U4 pad 53: (no net) -> RESET
- U4 pad 61: (no net) -> SD1_CD
Other:
- board text added: "20171130"
- board text removed: "20171129"

Commit message: 20171130
Parts:
- J1: footprint Connectors:PJ311_3.5mm_Jack -> mylib:pj311_3.5mm
- moved J1 4.02 mm to (104.1, 115.6), turned to 0 degrees
Changed lines of the file:
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@@
     (links 242)
     (no_connects 242)
-    (area 99.067143 64.335 219.074284 194.39)
+    (area 116.764999 67.234999 181.685001 137.235001)
     (thickness 1.6)
     (drawings 6)
@@
     )
   )
-  (module Connectors:PJ311_3.5mm_Jack (layer F.Cu)
-    (at 105.41 111.76 180)
-    (descr "PJ311 6pin SMD 3.5mm stereo headphones jack.")
-    (tags "headphones jack plug stereo 3.5mm PJ311")
-    (attr smd)
-    (fp_text reference J1 (at 0 -10.16 180) (layer F.SilkS)
-      (effects (font (size 1 1) (thickness 0.15)))
-    )
-    (fp_text value JACK_TRS_6PINS (at 0 7.17 180) (layer F.Fab)
-      (effects (font (size 1 1) (thickness 0.15)))
-    )
-    (fp_text user %R (at 0 0 180) (layer F.Fab)
-      (effects (font (size 1 1) (thickness 0.15)))
-    )
-    (fp_line (start -3.1 -5.5) (end -3.1 -6.9) (layer F.SilkS) (width 0.12))
-    (fp_line (start -3.1 -2.1) (end -3.1 -3.9) (layer F.SilkS) (width 0.12))
-    (fp_line (start -3.1 3.4) (end -3.1 -0.5) (layer F.SilkS) (width 0.12))
-    (fp_line (start 2.4 5.3) (end -3.1 5.3) (layer F.SilkS) (width 0.12))
-    (fp_line (start -3.1 5.3) (end -3.1 5) (layer F.SilkS) (width 0.12))
-    (fp_line (start 3.1 3.3) (end 3.1 3.9) (layer F.SilkS) (width 0.12))
-    (fp_line (start 3.1 -3.9) (end 3.1 1.7) (layer F.SilkS) (width 0.12))
-    (fp_line (start 3.1 -6.9) (end 3.1 -5.5) (layer F.SilkS) (width 0.12))
-    (fp_line (start -2.6 -6.9) (end -2.6 -8.9) (layer F.SilkS) (width 0.12))
-    (fp_line (start -2.6 -8.9) (end 2.6 -8.9) (layer F.SilkS) (width 0.12))
-    (fp_line (start 2.6 -8.9) (end 2.6 -6.9) (layer F.SilkS) (width 0.12))
-    (fp_line (start 2.6 -6.9) (end 3.1 -6.9) (layer F.SilkS) (width 0.12))
-    (fp_line (start -3.1 -6.9) (end -2.6 -6.9) (layer F.SilkS) (width 0.12))
-    (fp_line (start -3 5.2) (end 3 5.2) (layer F.Fab) (width 0.1))
-    (fp_line (start 3 5.2) (end 3 -6.8) (layer F.Fab) (width 0.1))
-    (fp_line (start 3 -6.8) (end 2.5 -6.8) (layer F.Fab) (width 0.1))
-    (fp_line (start 2.5 -6.8) (end 2.5 -8.8) (layer F.Fab) (width 0.1))
-    (fp_line (start 2.5 -8.8) (end -2.5 -8.8) (layer F.Fab) (width 0.1))
-    (fp_line (start -2.5 -8.8) (end -2.5 -6.8) (layer F.Fab) (width 0.1))
-    (fp_line (start -2.5 -6.8) (end -3 -6.8) (layer F.Fab) (width 0.1))
-    (fp_line (start -3 -6.8) (end -3 5.2) (layer F.Fab) (width 0.1))
-    (fp_line (start -5 -9.31) (end 5 -9.31) (layer F.CrtYd) (width 0.05))
-    (fp_line (start -5 -9.31) (end -5 5.94) (layer F.CrtYd) (width 0.05))
-    (fp_line (start 5 5.94) (end 5 -9.31) (layer F.CrtYd) (width 0.05))
-    (fp_line (start -5 5.94) (end 5 5.94) (layer F.CrtYd) (width 0.05))
-    (pad 6 smd rect (at -3.5 4.2 180) (size 2 1.5) (layers F.Cu F.Paste F.Mask)
-      (net 11 OUTR))
-    (pad 3 smd rect (at -3.5 -1.3 180) (size 2 1.5) (layers F.Cu F.Paste F.Mask))
-    (pad 1 smd rect (at -3.5 -4.7 180) (size 2 1.5) (layers F.Cu F.Paste F.Mask)
-      (net 2 GND))
-    (pad 5 smd rect (at 3.5 4.7 180) (size 2 1.5) (layers F.Cu F.Paste F.Mask)
-      (net 10 OUTL))
-    (pad 4 smd rect (at 3.5 2.5 180) (size 2 1.5) (layers F.Cu F.Paste F.Mask)
-      (net 2 GND))
-    (pad "" np_thru_hole circle (at 0 -4.3 180) (size 1.5 1.5) (drill 1.5) (layers *.Cu *.Mask F.SilkS))
-    (pad "" np_thru_hole circle (at 0 2.7 180) (size 1.5 1.5) (drill 1.5) (layers *.Cu *.Mask F.SilkS))
-    (pad 2 smd rect (at 3.5 -4.7 180) (size 2 1.5) (layers F.Cu F.Paste F.Mask)
-      (net 55 MUTE))
-  )
   (module Resistors_SMD:R_2010_HandSoldering (layer F.Cu)
     (at 158.75 71.12)
@@
     )
   )
+  (module mylib:pj311_3.5mm (layer F.Cu)
+    (at 104.14 115.57)
+    (descr "PJ311 6pin SMD 3.5mm stereo headphones jack.")
+    (tags "headphones jack plug stereo 3.5mm PJ311")
+    (attr smd)
+    (fp_text reference J1 (at 0 -10.16) (layer F.SilkS)
+      (effects (font (size 1 1) (thickness 0.15)))
+    )
+    (fp_text value JACK_TRS_6PINS (at 0 7.17) (layer F.Fab)
+      (effects (font (size 1 1) (thickness 0.15)))
+    )
+    (fp_line (start -3.1 3.3) (end -3.1 5.3) (layer F.SilkS) (width 0.12))
+    (fp_line (start -3.1 5.3) (end 3.1 5.3) (layer F.SilkS) (width 0.12))
+    (fp_line (start 3.1 5.3) (end 3.1 3.35) (layer F.SilkS) (width 0.12))
+    (fp_line (start -3.1 -0.5) (end -3.1 1.7) (layer F.SilkS) (width 0.12))
+    (fp_text user %R (at 0 0) (layer F.Fab)
+      (effects (font (size 1 1) (thickness 0.15)))
+    )
+    (fp_line (start -3.1 -5.5) (end -3.1 -6.9) (layer F.SilkS) (width 0.12))
+    (fp_line (start -3.1 -2.1) (end -3.1 -3.9) (layer F.SilkS) (width 0.12))
+    (fp_line (start 3.1 -3.9) (end 3.1 1.7) (layer F.SilkS) (width 0.12))
+    (fp_line (start 3.1 -6.9) (end 3.1 -5.5) (layer F.SilkS) (width 0.12))
+    (fp_line (start -2.6 -6.9) (end -2.6 -8.9) (layer F.SilkS) (width 0.12))
+    (fp_line (start -2.6 -8.9) (end 2.6 -8.9) (layer F.SilkS) (width 0.12))
+    (fp_line (start 2.6 -8.9) (end 2.6 -6.9) (layer F.SilkS) (width 0.12))
+    (fp_line (start 2.6 -6.9) (end 3.1 -6.9) (layer F.SilkS) (width 0.12))
+    (fp_line (start -3.1 -6.9) (end -2.6 -6.9) (layer F.SilkS) (width 0.12))
+    (fp_line (start -3 5.2) (end 3 5.2) (layer F.Fab) (width 0.1))
+    (fp_line (start 3 5.2) (end 3 -6.8) (layer F.Fab) (width 0.1))
+    (fp_line (start 3 -6.8) (end 2.5 -6.8) (layer F.Fab) (width 0.1))
+    (fp_line (start 2.5 -6.8) (end 2.5 -8.8) (layer F.Fab) (width 0.1))
+    (fp_line (start 2.5 -8.8) (end -2.5 -8.8) (layer F.Fab) (width 0.1))
+    (fp_line (start -2.5 -8.8) (end -2.5 -6.8) (layer F.Fab) (width 0.1))
+    (fp_line (start -2.5 -6.8) (end -3 -6.8) (layer F.Fab) (width 0.1))
+    (fp_line (start -3 -6.8) (end -3 5.2) (layer F.Fab) (width 0.1))
+    (fp_line (start -5 -9.31) (end 5 -9.31) (layer F.CrtYd) (width 0.05))
+    (fp_line (start -5 -9.31) (end -5 5.94) (layer F.CrtYd) (width 0.05))
+    (fp_line (start 5 5.94) (end 5 -9.31) (layer F.CrtYd) (width 0.05))
+    (fp_line (start -5 5.94) (end 5 5.94) (layer F.CrtYd) (width 0.05))
+    (pad 6 smd rect (at 3.5 2.5) (size 2 1.5) (layers F.Cu F.Paste F.Mask)
+      (net 11 OUTR))
+    (pad 3 smd rect (at -3.5 -1.3) (size 2 1.5) (layers F.Cu F.Paste F.Mask))
+    (pad 1 smd rect (at -3.5 -4.7) (size 2 1.5) (layers F.Cu F.Paste F.Mask)
+      (net 2 GND))
+    (pad 5 smd rect (at -3.5 2.5) (size 2 1.5) (layers F.Cu F.Paste F.Mask)
+      (net 10 OUTL))
+    (pad 4 smd rect (at 3.5 -1.3) (size 2 1.5) (layers F.Cu F.Paste F.Mask)
+      (net 2 GND))
+    (pad "" thru_hole circle (at 0 -4.3) (size 1.5 1.5) (drill 1) (layers *.Cu *.Mask))
+    (pad "" thru_hole circle (at 0 2.7) (size 1.5 1.5) (drill 1) (layers *.Cu *.Mask))
+    (pad 2 smd rect (at 3.5 -4.7) (size 2 1.5) (layers F.Cu F.Paste F.Mask)
+      (net 55 MUTE))
+  )
   (gr_line (start 116.84 137.16) (end 116.84 67.31) (angle 90) (layer Edge.Cuts) (width 0.15))

Commit message: 20171201
Parts:
- BAT1, P6: footprint Connectors_Molex:Molex_SPOX-5267_22-03-5035_03x2.54mm_Straight -> Connectors:GS3
- C1, C10, C11, C12, C3, C4, C5, C6, C7, C8, R1, R10, R11, R12, R13, R14, R15, R16, R17, R18, R19, R2, R20, R21, R22, R23, R24, R25, R26, R27, R28, R3, R4, R5, R6, R7, R8, R9: moved to B.Cu
- LS1, LS2: footprint Resistors_SMD:R_2010_HandSoldering -> Connectors:GS2
- U3: footprint mylib:fpc-45pin-0.5mm -> mylib:fpc-45pin-0.5mm-down
- moved R4 84.5 mm to (121.9, 133.3), turned to 90 degrees
- moved C9 72.8 mm to (129.5, 127.0), turned to 90 degrees
- moved SW9 71.9 mm to (172.7, 69.8)
- moved C3 71.4 mm to (147.3, 123.2)
- moved C6 70.0 mm to (119.4, 109.2), turned to 270 degrees
- moved C8 69.2 mm to (142.2, 123.2)
- moved C12 67.7 mm to (160.0, 133.3), turned to 270 degrees
- moved C1 64.5 mm to (157.5, 133.3), turned to 90 degrees
- moved R8 63.1 mm to (171.4, 104.1)
- moved LS1 61.0 mm to (123.2, 120.7)
- moved C2 60.7 mm to (139.7, 128.3)
- moved C7 60.3 mm to (128.3, 78.7), turned to 90 degrees
- moved R5 60.3 mm to (171.4, 109.2)
- moved C11 59.5 mm to (153.7, 128.3)
- moved R25 59.2 mm to (166.4, 101.6)
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
Commit message: 20171204
Parts:
- P4: footprint Connectors:USB_Micro-B -> Connectors:USB_Mini-B
- moved P4 58.4 mm to (161.3, 133.3), turned to 90 degrees
- moved J1 55.9 mm to (132.1, 129.5), turned to 180 degrees
- moved C9 47.0 mm to (176.5, 128.3), turned to 270 degrees
- moved SW2 19.1 mm to (130.8, 69.8), turned to 0 degrees
- moved C2 10.9 mm to (129.5, 124.5)
- moved U2 1.27 mm to (121.9, 129.5)
- moved CON1 1.27 mm to (179.1, 123.2)
- moved CON2 1.27 mm to (179.1, 102.9)

Commit message: 20171207
Parts:
- BAT1, P6: footprint Connectors:GS3 -> GS3
- C1, C10, C11, C12, C3, C4, C5, C6, C7, C8: footprint Capacitors_SMD:C_0603_HandSoldering -> MyFT_C_0603; moved to F.Cu
- C2, C9: footprint Capacitors_SMD:C_0603_HandSoldering -> MyFT_C_0603
- CON1, CON2: footprint mylib:microsd -> MyFT_MicroSD
- J1: footprint mylib:pj311_3.5mm -> MyFT_PJ311_3.5mm
- LS1, LS2: footprint Connectors:GS2 -> GS2
- P1: footprint mylib:volumn -> MyFT_Volumn
- P4: footprint Connectors:USB_Mini-B -> MyFT_MiniUSB_B
- Q1: footprint TO_SOT_Packages_SMD:SOT-23-5_HandSoldering -> MyFT_SOT-223
- R1, R10, R11, R12, R13, R14, R15, R16, R17, R18, R19, R2, R20, R21, R22, R23, R24, R25, R26, R27, R28, R3, R4, R5, R6, R7, R8, R9: footprint Resistors_SMD:R_0603_HandSoldering -> MyFT_R_0603; moved to F.Cu
- SW1, SW10, SW2, SW9: footprint Buttons_Switches_THT:SW_PUSH_6mm -> MyFT_SW_PUSH_6mm
- SW11, SW5, SW6: footprint mylib:dpad-h -> MyFT_DPAD_LR
- SW12, SW3, SW4: footprint mylib:dpad-v -> MyFT_DPAD_TB
- SW13: footprint mylib:dpad-h -> MyFT_DPAD_TB
- SW14: footprint mylib:dpad-v -> MyFT_DPAD_LR
- SW7, SW8: footprint Buttons_Switches_SMD:SW_SPST_TL3342 -> MyFT_SW_SPST_TL3342
- U1: footprint Housings_SSOP:TSSOP-20_4.4x6.5mm_Pitch0.65mm -> MyFT_TSSOP-20_4.4x6.5mm_Pitch0.65mm
- U2: footprint Housings_SSOP:SOP-16_4.4x10.4mm_Pitch1.27mm -> MyFT_SOP-16_4.4x10.4mm_Pitch1.27mm
- U3: footprint mylib:fpc-45pin-0.5mm-down -> MyFT_FPC_45_0.5mm
- U4: footprint mylib:cm3354 -> MyFT_CM3354
- U5: footprint mylib:sc-70-5 -> MyFT_SC-70-5
- moved R17 227.1 mm to (345.4, 121.9), turned to 0 degrees
- moved R20 215.0 mm to (337.8, 120.7)
- moved C5 209.7 mm to (327.7, 123.2), turned to 0 degrees
- moved R18 197.3 mm to (321.3, 114.3), turned to 0 degrees
- moved R2 193.1 mm to (334.0, 123.2)
- moved R21 193.1 mm to (316.2, 113.0)
- moved C8 185.5 mm to (327.7, 128.3)
- moved R10 184.2 mm to (344.2, 118.1)
- moved R12 184.1 mm to (307.3, 116.8), turned to 0 degrees
- moved R4 183.3 mm to (304.8, 120.7), turned to 0 degrees
- moved R25 176.9 mm to (341.6, 125.7)
- moved R27 175.3 mm to (309.9, 121.9)
- moved Q1 169.2 mm to (328.9, 115.6)
- moved R6 166.4 mm to (285.8, 109.2), turned to 0 degrees
- moved R14 165.3 mm to (317.5, 116.8)
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Connections:
- net +3V3 renamed +3.3V
- SW4 pad 1: (no net) -> DOWN
- SW4 pad 2: (no net) -> GND
Other:
- board size 64.8 x 69.8 mm -> 64.8 x 69.9 mm
- net class Default: clearance 0.2 -> 0.254; trace_width 0.25 -> 0.254; via_dia 0.6 -> 0.889; via_drill 0.4 -> 0.635
- rule pad_to_mask_clearance: 0.2 -> 0
- rule trace_clearance: 0.2 -> 0.254
- rule trace_min: 0.2 -> 0.254
- rule via_min_drill: 0.3 -> 0.508
- rule via_min_size: 0.4 -> 0.889
- board text removed: "20171130"
- board text removed: "Handmade01"

Commit message: 20171208
Parts:
- Q1: footprint MyFT_SOT-223 -> MyFT_SOT-23_Handsoldering
- SW1: value POWER -> Power; footprint MyFT_SW_PUSH_6mm -> MyFT_TS-026-3
- SW10, SW2, SW9: footprint MyFT_SW_PUSH_6mm -> MyFT_TS-026-3
- moved R17 113.0 mm to (246.4, 176.3)
- moved R10 108.9 mm to (252.7, 177.3)
- moved R20 94.9 mm to (260.4, 175.5)
- moved R25 91.3 mm to (266.4, 177.5)
- moved P6 88.2 mm to (286.3, 156.7), turned to 270 degrees
- moved C3 79.3 mm to (224.3, 174.2)
- moved R22 79.2 mm to (231.1, 175.0)
- moved R18 78.6 mm to (272.3, 175.8)
- moved R13 78.4 mm to (264.9, 172.5)
- moved R2 76.4 mm to (277.1, 174.2)
- moved LS1 75.2 mm to (211.8, 114.6)
- moved R21 71.4 mm to (273.8, 170.4)
- moved SW1 71.2 mm to (244.6, 166.9), turned to 90 degrees
- moved U5 70.9 mm to (242.1, 112.0), turned to 270 degrees
- moved Q1 68.1 mm to (260.9, 112.5), turned to 180 degrees
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Other:
- board size 64.8 x 69.9 mm -> 64.8 x 70.1 mm

Commit message: 20171208
Parts:
- moved BAT1 95.9 mm to (146.6, 79.5)
- moved C1 95.9 mm to (105.4, 131.3)
- moved C3 95.9 mm to (134.1, 141.7)
- moved C5 95.9 mm to (189.0, 137.7)
- moved C6 95.9 mm to (179.8, 92.7)
- moved CON1 95.9 mm to (170.2, 133.6)
- moved LS1 95.9 mm to (121.7, 82.0)
- moved P1 95.9 mm to (142.7, 131.3)
- moved Q1 95.9 mm to (170.7, 80.0)
- moved R12 95.9 mm to (179.8, 129.3)
- moved R13 95.9 mm to (174.8, 140.0)
- moved R18 95.9 mm to (182.1, 143.3)
- moved R19 95.9 mm to (194.3, 120.9)
- moved R20 95.9 mm to (170.2, 143.0)
- moved R21 95.9 mm to (183.6, 137.9)
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