File: handmade01/main.kicad_pcb (KiCad board)
At the start: 2 copper layers, 64.8 x 70.1 mm, 71 parts, among them CON1 MicroSD, CON2 MicroSD, J1 JACK_TRS_6PINS, P1 VOLUMN, P4 USB_OTG, P6 UART_DEBUG, Q1 1AM, SW1 Power, SW10 R, SW11 A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

Commit message: 20171215
Routing:
- net START: track 18.1 -> 26.3 mm
- net SD1_DAT3: track 64.2 -> 71.6 mm
- net SD1_DAT1: track 81.6 -> 88.4 mm
- net SD1_DAT0: track 76.3 -> 82.9 mm
- net SD1_CLK: track 78.5 -> 81.5 mm
- net SD1_CMD: track 74.4 -> 71.7 mm
- net DOWN: track 26.7 -> 28.9 mm
- net SD1_DAT2: track 70.8 -> 69.5 mm

Commit message: 20171216
Routing:
- net LCD_SDO: track 0.00 -> 54.5 mm, vias 0 -> 2
- net LCD_SDI: track 2.70 -> 55.3 mm, vias 1 -> 2
- net LCD_CS: track 0.00 -> 52.0 mm, vias 0 -> 2
- net LCD_SCL: track 0.00 -> 50.6 mm, vias 0 -> 2
- net SD1_DAT1: track 88.4 -> 80.1 mm
- net SD1_CLK: track 81.5 -> 76.8 mm
- net SD1_CMD: track 71.7 -> 75.6 mm
- net UP: track 14.9 -> 18.1 mm
- net SD1_DAT0: track 82.9 -> 81.0 mm
- net SD1_DAT3: track 71.6 -> 70.0 mm
- net SD1_DAT2: track 69.5 -> 70.7 mm
- net AUDIO_BCK: track 22.0 -> 23.0 mm

Commit message: 20171216
Parts:
- R11, R15, R17, R19, R21, R23, R25, R29, R30, R5, R6, R7, R8, R9: moved to F.Cu
- moved R21 70.1 mm to (128.4, 79.2), turned to 270 degrees
- moved R30 32.1 mm to (135.8, 123.4)
- moved R11 28.0 mm to (119.8, 107.9), turned to 0 degrees
- moved R9 20.8 mm to (111.4, 116.3)
- moved R19 17.7 mm to (165.2, 119.2), turned to 180 degrees
- moved R17 16.6 mm to (161.4, 120.1), turned to 180 degrees
- moved R15 16.5 mm to (156.3, 124.5), turned to 270 degrees
- moved R25 16.2 mm to (169.8, 119.9), turned to 180 degrees
- moved R8 16.1 mm to (115.5, 119.7), turned to 180 degrees
- moved R23 15.8 mm to (172.8, 120.0)
- moved R5 15.7 mm to (113.0, 120.1), turned to 270 degrees
- moved R6 15.7 mm to (111.4, 120.1), turned to 270 degrees
- moved R7 14.6 mm to (117.5, 121.2), turned to 0 degrees
- moved R29 12.4 mm to (128.7, 126.6)
- moved R4 0.88 mm to (141.2, 72.7)
Routing:
- net L: track 0.00 -> 77.4 mm
- net INL: track 0.00 -> 66.9 mm, vias 0 -> 1
- net UART_RX: track 0.00 -> 62.7 mm, vias 0 -> 2
- net UART_TX: track 0.00 -> 62.6 mm, vias 0 -> 2
- net OUTL: track 1.91 -> 63.8 mm, vias 0 -> 1
- net INR: track 0.00 -> 60.6 mm, vias 0 -> 1
- net LCD_RESET: track 0.00 -> 53.5 mm, vias 0 -> 2
- net OUTR: track 1.66 -> 53.0 mm, vias 0 -> 1
- net MUTE: track 0.00 -> 42.4 mm, vias 0 -> 2
- net R: track 0.00 -> 38.0 mm
- net SD0_DAT1: track 48.8 -> 35.2 mm, vias 1 -> 0
- net LED_K: track 0.00 -> 10.5 mm
- net BAT_+: track 0.00 -> 9.81 mm
- net SD0_DAT0: track 41.5 -> 32.3 mm, vias 1 -> 0
- net SD0_DAT3: track 47.2 -> 38.2 mm
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
Commit message: 20171216
Parts:
- moved C9 17.8 mm to (171.4, 102.4)
- moved R25 15.7 mm to (156.0, 127.4), turned to 0 degrees
- moved R14 14.2 mm to (133.7, 127.1), turned to 0 degrees
- moved C5 4.00 mm to (114.1, 90.8), turned to 0 degrees
- moved R23 3.59 mm to (169.4, 121.1), turned to 180 degrees
- moved R18 2.88 mm to (155.1, 132.4), turned to 180 degrees
- moved R3 2.58 mm to (172.7, 81.5)
- moved Q1 2.21 mm to (170.0, 82.1), turned to 270 degrees
- moved R19 1.97 mm to (165.7, 121.1)
- moved R16 1.29 mm to (132.3, 130.6), turned to 0 degrees
- moved C10 1.14 mm to (163.1, 114.7)
- moved LS1 1.02 mm to (121.3, 81.3)
- moved LS2 1.02 mm to (111.4, 81.3)
- moved R17 1.02 mm to (161.4, 121.1)
- moved C1 0.50 mm to (169.9, 102.4)
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Routing:
- net OUTR: track 53.0 -> 112.5 mm, vias 1 -> 2
- net LCD_RESET: track 53.5 -> 2.14 mm, vias 2 -> 1
- net SD1_CD: track 6.06 -> 55.3 mm, vias 0 -> 2
- net OUTL: track 63.8 -> 111.5 mm, vias 1 -> 2
- net USB_DM: track 0.00 -> 33.0 mm, vias 0 -> 2
- net GND: track 17.2 -> 48.4 mm
- net USB_DP: track 0.00 -> 30.4 mm, vias 0 -> 2
- net RIGHT: track 12.6 -> 32.8 mm, vias 1 -> 3
- net SD1_DAT1: track 88.1 -> 80.2 mm
- net LED_PWM: track 37.5 -> 44.1 mm
- net LED_K: track 10.5 -> 4.06 mm
- net AUDIO_BCK: track 23.0 -> 29.2 mm
- net LCD_DB6: track 31.7 -> 37.2 mm
- net AUDIO_MUTE: track 12.0 -> 7.39 mm, vias 2 -> 0
- net SELECT: track 32.6 -> 37.1 mm, vias 2 -> 1
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
Commit message: 20171216
Parts:
- moved P6 51.3 mm to (111.4, 109.3), turned to 0 degrees
- moved Q1 1.40 mm to (170.1, 80.7)
- moved R20 0.51 mm to (173.5, 75.4)
- moved R1 0.32 mm to (174.4, 108.3)
- moved R21 0.18 mm to (128.3, 79.4)
- moved R2 0.13 mm to (172.9, 105.7)
- moved C8 0.13 mm to (172.9, 102.0)
Routing:
- net UART_RX: track 63.2 -> 0.00 mm, vias 2 -> 0
- net UART_TX: track 63.1 -> 0.00 mm, vias 2 -> 0
- net LCD_RESET: track 2.14 -> 52.2 mm, vias 1 -> 2
- net USB_DM: track 33.0 -> 0.00 mm, vias 2 -> 0
- net USB_DP: track 30.4 -> 0.00 mm, vias 2 -> 0
- net GND: track 48.4 -> 28.6 mm
- net LCD_SDO: track 60.2 -> 71.2 mm
- net LCD_DB6: track 37.2 -> 27.0 mm
- net BAT_+: track 9.81 -> 0.00 mm
- net X: track 33.3 -> 27.3 mm
- net LCD_DB13: track 34.9 -> 39.7 mm
- net RTC_+: track 4.69 -> 0.00 mm
- net LCD_DB10: track 33.7 -> 38.4 mm
- net BAT_T: track 3.73 -> 0.00 mm
- net LCD_DB11: track 29.4 -> 32.7 mm
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
Commit message: 20171217
Parts:
- moved R17 54.2 mm to (126.7, 79.4), turned to 270 degrees
- moved R15 46.1 mm to (121.5, 94.2)
- moved R9 13.5 mm to (120.5, 106.3), turned to 0 degrees
- moved R8 12.3 mm to (117.8, 107.6), turned to 270 degrees
- moved R5 11.6 mm to (121.5, 112.2)
- moved R7 10.9 mm to (116.8, 110.3)
- moved R29 9.46 mm to (121.2, 120.8), turned to 180 degrees
- moved P6 5.59 mm to (111.5, 103.7)
- moved R25 2.17 mm to (154.9, 125.5), turned to 90 degrees
- moved R14 1.34 mm to (133.8, 128.4)
- moved R6 1.18 mm to (112.3, 120.8), turned to 0 degrees
- moved R18 0.97 mm to (154.9, 131.4), turned to 270 degrees
- moved R11 0.72 mm to (120.5, 108.1)
- moved BAT1 0.60 mm to (147.1, 79.2)
- moved R4 0.51 mm to (141.2, 73.2)
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Routing:
- net GND: track 28.6 -> 586.5 mm, vias 0 -> 29
- net +3.3V: track 14.4 -> 363.5 mm, vias 0 -> 29
- net POWER: track 0.00 -> 106.8 mm, vias 0 -> 6
- net UART_TX: track 0.00 -> 41.6 mm, vias 0 -> 2
- net UART_RX: track 0.00 -> 39.4 mm, vias 0 -> 2
- net USB_DM: track 0.00 -> 31.6 mm
- net USB_DP: track 0.00 -> 29.0 mm
- net +5V: track 0.00 -> 17.3 mm
- net SD0_CLK: track 35.6 -> 21.3 mm, vias 2 -> 0
- net SD0_CMD: track 39.8 -> 26.9 mm
- net BAT_+: track 0.00 -> 12.8 mm
- net SD0_DAT3: track 40.0 -> 28.8 mm, vias 2 -> 0
- net SD0_CD: track 21.4 -> 12.3 mm, vias 2 -> 0
- net SD0_DAT2: track 42.6 -> 34.2 mm
- net R: track 38.0 -> 46.1 mm, vias 0 -> 1
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
Commit message: 20171217
Routing:
- added copper zone on B.Cu, net GND
- added copper zone on F.Cu, net GND
Changed lines of the file:
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@@
   (page A4)
   (layers
-    (15 F.Cu signal)
-    (0 B.Cu signal)
-    (16 B.Adhes user)
-    (17 F.Adhes user)
-    (18 B.Paste user)
-    (19 F.Paste user)
-    (20 B.SilkS user)
-    (21 F.SilkS user)
-    (22 B.Mask user)
-    (23 F.Mask user)
-    (24 Dwgs.User user)
-    (25 Cmts.User user)
-    (26 Eco1.User user)
-    (27 Eco2.User user)
+    (15 F.Cu signal hide)
+    (0 B.Cu signal hide)
+    (16 B.Adhes user hide)
+    (17 F.Adhes user hide)
+    (18 B.Paste user hide)
+    (19 F.Paste user hide)
+    (20 B.SilkS user hide)
+    (21 F.SilkS user hide)
+    (22 B.Mask user hide)
+    (23 F.Mask user hide)
+    (24 Dwgs.User user hide)
+    (25 Cmts.User user hide)
+    (26 Eco1.User user hide)
+    (27 Eco2.User user hide)
     (28 Edge.Cuts user)
   )
@@
     (pad_to_mask_clearance 0)
     (aux_axis_origin 0 0)
-    (visible_elements 7FFFFFEF)
+    (visible_elements 7FFFFFFF)
     (pcbplotparams
       (layerselection 536838145)
@@
   (segment (start 134.62 122.494) (end 134.62 120.0731) (width 0.18) (layer F.Cu) (net 87))
   (segment (start 134.62 120.0731) (end 134.6098 120.0629) (width 0.18) (layer F.Cu) (net 87))
+  (zone (net 12) (net_name GND) (layer B.Cu) (hatch edge 0.508)
+    (connect_pads (clearance 0.18))
+    (min_thickness 0.18)
+    (fill (arc_segments 16) (thermal_gap 0.2) (thermal_bridge_width 0.2))
+    (polygon
+      (pts
+        (xy 175.26 137.668) (xy 110.49 137.668) (xy 110.49 73.152) (xy 130.302 73.152) (xy 130.302 67.564)
+        (xy 155.194 67.564) (xy 155.194 73.152) (xy 175.26 73.152) (xy 175.26 77.724) (xy 173.736 77.724)
+        (xy 173.736 101.6) (xy 175.26 101.6)
+      )
+    )
+  )
+  (zone (net 12) (net_name GND) (layer F.Cu) (hatch edge 0.508)
+    (connect_pads (clearance 0.18))
+    (min_thickness 0.18)
+    (fill (arc_segments 16) (thermal_gap 0.2) (thermal_bridge_width 0.2))
+    (polygon
+      (pts
+        (xy 175.26 137.668) (xy 110.49 137.668) (xy 110.49 73.152) (xy 130.302 73.152) (xy 130.302 67.564)
+        (xy 155.194 67.564) (xy 155.194 73.152) (xy 175.26 73.152) (xy 175.26 77.724) (xy 173.736 77.724)
+        (xy 173.736 101.6) (xy 175.26 101.6)
+      )
+    )
+  )
 )

Commit message: 20171217
Parts:
- moved R20 9.01 mm to (164.6, 73.9), turned to 0 degrees
Routing:
- net GND: track 586.5 -> 600.7 mm
- net +3.3V: track 363.5 -> 373.1 mm
- net L: track 83.9 -> 88.4 mm, vias 2 -> 1
- net +5V: track 17.3 -> 15.2 mm
- added copper zone on F.Cu, net +5V
- added copper zone on F.Cu, net BAT_+
- added copper zone on F.Cu, net BAT_T
Other:
- outline, holes or cut-outs redrawn
- board text added: "Handmade01 Steward 20171217"
- board text removed: "Handmade01 Steward 20171212"
