File: handmade01/main.sch (KiCad schematic (older format))
At the start: 2 parts

Commit message: 20171106
Parts:
- removed P?: USB_OTG, symbol USB_OTG
- removed U?: CM3354, symbol CM3354
- added C1: 10uF, symbol C
- added C10, C4, C5, C6, C9: 0.1uF, symbol C
- added C11, C12: 1uF, symbol C
- added C2, C3: 2.2uF, symbol C
- added C7, C8: 2.2nF, symbol C
- added CON1: SD0, symbol Micro_SD_Card
- added CON2: SD1, symbol Micro_SD_Card
- added LS?: SPEAKER_L, symbol Speaker
- added LS?: SPEAKER_R, symbol Speaker
- added P1: VOLUMN, symbol CONN_01X05
- added P4: USB_OTG, symbol USB_OTG
- added P5: BATTERY, symbol CONN_01X03
- added P6: UART_DEBUG, symbol CONN_01X03
- added Q1: 1AM, symbol Q_NPN_BCE
- added R1, R2: 10K, symbol R
- added R3: 4.7K, symbol R
- added RN1: SD0_4.7K, Resistors_ThroughHole:Resistor_Array_SIP7, symbol R_Network06
- added RN2: SD1_4.7K, Resistors_ThroughHole:Resistor_Array_SIP7, symbol R_Network06
- added RN3: GAMEPAD_4.7K, Resistors_ThroughHole:Resistor_Array_SIP13, symbol R_Network12
- added SW1: POWER, symbol SW_Push_Dual_x2
- added SW10: R, symbol SW_Push_Dual_x2
- added SW11: A, symbol SW_Push_Dual_x2
- added SW12: B, symbol SW_Push_Dual_x2
- added SW13: X, symbol SW_Push_Dual_x2
- added SW14: Y, symbol SW_Push_Dual_x2
- added SW2: RESET, symbol SW_Push_Dual_x2
- added SW3: UP, symbol SW_Push_Dual_x2
- added SW4: DOWN, symbol SW_Push_Dual_x2
- added SW5: LEFT, symbol SW_Push_Dual_x2
- added SW6: RIGHT, symbol SW_Push_Dual_x2
- added SW7: SELECT, symbol SW_Push_Dual_x2
- added SW8: START, symbol SW_Push_Dual_x2
- added SW9: L, symbol SW_Push_Dual_x2
- added U1: PCM5102A, symbol PCM5102A
- added U2: PAM8403, symbol PAM8403
- added U3: IPS_2.4_240x320_ST7789V, symbol IPS_2.4_240x320_ST7789V
- added U4: CM3354, symbol CM3354
- added U5: TPS71718, symbol TPS71718
Connections:
- net labels added: A, AUDIO_BCK, AUDIO_DIN, AUDIO_LRCK, AUDIO_MUTE, B, BAT_+, BAT_-, BAT_T, DOWN, INL, INR, L, LCD_CS, LCD_DB0, LCD_DB1, LCD_DB10, LCD_DB11, LCD_DB12, LCD_DB13, LCD_DB14, LCD_DB15, LCD_DB2, LCD_DB3, LCD_DB4, LCD_DB5, LCD_DB6, LCD_DB7, LCD_DB8, LCD_DB9, LCD_ENABLE, LCD_HSYNC, LCD_PCLK, LCD_RESET, LCD_SCL, LCD_SDI, LCD_SDO, LCD_VSYNC, LED_K, LED_PWM, LEFT, OUTL, OUTR, OUT_L+, OUT_L-, OUT_R+, OUT_R-, POWER, R, RESET, RIGHT, RTC_+, SD0_CD, SD0_CLK, SD0_CMD, SD0_DAT0, SD0_DAT1, SD0_DAT2, SD0_DAT3, SD1_CLK, SD1_CMD, SD1_DAT0, SD1_DAT1, SD1_DAT2, SD1_DAT3, SDO_CLK, SELECT, START, UART_RX, UART_TX, UP, USB_DM, USB_DP, X, Y
- wire segments 0 -> 33
Other:
- note added: "20171106"
- note removed: "20171101"

Commit message: 20171106
Parts:
- P4: symbol USB_OTG -> USB_OTG-RESCUE-main
Changed lines of the file:
@@
 EESchema Schematic File Version 2
+LIBS:main-rescue
 LIBS:power
 LIBS:device
@@
 $EndComp
 $Comp
-L USB_OTG P4
+L USB_OTG-RESCUE-main P4
 U 1 1 59FFDB87
 P 6400 9800

Commit message: 20171109
Parts:
- gave numbers to parts that had none: 2

Commit message: 20171109
Parts:
- removed CON1: SD0, symbol Micro_SD_Card
- removed CON2: SD1, symbol Micro_SD_Card
- removed P5: BATTERY, symbol CONN_01X03
- added BAT1: BAT, symbol BAT
- added CON1, CON2: MicroSD, symbol MicroSD
Connections:
- net labels added: SD1_CD
- net labels removed: BAT_-, SDO_CLK
- wire segments 33 -> 34
- no-connect marks 0 -> 34
Other:
- note added: "20171109"
- note removed: "20171106"
Changed lines of the file:
@@
 handmade01
 Text Notes 13000 11050 0    60   ~ 12
-20171106
+20171109
 $Comp
 L +5V #PWR05
@@
 Text GLabel 7450 8650 3    60   Input ~ 0
 BAT_T
-$Comp
-L CONN_01X03 P5
-U 1 1 59FFDCE7
-P 7500 9750
-F 0 "P5" H 7500 9950 50  0000 C CNN
-F 1 "BATTERY" V 7600 9750 50  0000 C CNN
-F 2 "" H 7500 9750 50  0000 C CNN
-F 3 "" H 7500 9750 50  0000 C CNN
-	1    7500 9750
-	0    -1   -1   0
-$EndComp
-Text GLabel 7400 9950 3    60   Input ~ 0
+Text GLabel 7500 9850 1    60   Input ~ 0
 BAT_+
-Text GLabel 7500 9950 3    60   Input ~ 0
+Text GLabel 7450 10150 3    60   Input ~ 0
 BAT_T
-Text GLabel 7600 9950 3    60   Input ~ 0
-BAT_-
 Text GLabel 7050 8650 3    60   Input ~ 0
 RTC_+
@@
 Text GLabel 5350 6350 0    60   Input ~ 0
 LCD_DB9
-Text GLabel 5350 6450 0    60   Input ~ 0
+Text GLabel 5350 6450 0    60   BiDi ~ 0
 LCD_DB12
 Text GLabel 5350 6550 0    60   Input ~ 0
@@
 	0    -1   -1   0
 $EndComp
-Text GLabel 11100 1750 3    60   Input ~ 0
-GND
 Text GLabel 11200 1750 3    60   Input ~ 0
 UART_TX
@@
 SD0_CD
 $Comp
-L Micro_SD_Card CON1
-U 1 1 5A00A9A2
-P 12950 5150
-F 0 "CON1" H 12300 5750 50  0000 C CNN
-F 1 "SD0" H 13600 5750 50  0000 R CNN
-F 2 "" H 14100 5450 50  0000 C CNN
-F 3 "" H 12950 5150 50  0000 C CNN
-	1    12950 5150
-	0    -1   -1   0
-$EndComp
-$Comp
-L Micro_SD_Card CON2
-U 1 1 5A00AA44
-P 14300 5150
-F 0 "CON2" H 13650 5750 50  0000 C CNN
-F 1 "SD1" H 14950 5750 50  0000 R CNN
-F 2 "" H 15450 5450 50  0000 C CNN
-F 3 "" H 14300 5150 50  0000 C CNN
-	1    14300 5150
-	0    -1   -1   0
-$EndComp
-$Comp
 L GND #PWR025
 U 1 1 5A00AADD
-P 13150 6050
-F 0 "#PWR025" H 13150 5800 50  0001 C CNN
-F 1 "GND" H 13150 5900 50  0000 C CNN
-F 2 "" H 13150 6050 50  0000 C CNN
-F 3 "" H 13150 6050 50  0000 C CNN
-	1    13150 6050
+P 12750 6150
+F 0 "#PWR025" H 12750 5900 50  0001 C CNN
+F 1 "GND" H 12750 6000 50  0000 C CNN
+F 2 "" H 12750 6150 50  0000 C CNN
+F 3 "" H 12750 6150 50  0000 C CNN
+	1    12750 6150
 	1    0    0    -1
 $EndComp
@@
 L GND #PWR026
 U 1 1 5A00AB1B
-P 14500 6050
-F 0 "#PWR026" H 14500 5800 50  0001 C CNN
-F 1 "GND" H 14500 5900 50  0000 C CNN
-F 2 "" H 14500 6050 50  0000 C CNN
-F 3 "" H 14500 6050 50  0000 C CNN
-	1    14500 6050
+P 14300 6150
+F 0 "#PWR026" H 14300 5900 50  0001 C CNN
+F 1 "GND" H 14300 6000 50  0000 C CNN
+F 2 "" H 14300 6150 50  0000 C CNN
+F 3 "" H 14300 6150 50  0000 C CNN
+	1    14300 6150
 	1    0    0    -1
 $EndComp
@@
 L +3.3V #PWR027
 U 1 1 5A00AB59
-P 14300 6050
-F 0 "#PWR027" H 14300 5900 50  0001 C CNN
-F 1 "+3.3V" H 14300 6190 50  0000 C CNN
-F 2 "" H 14300 6050 50  0000 C CNN
-F 3 "" H 14300 6050 50  0000 C CNN
-	1    14300 6050
+P 14100 6150
+F 0 "#PWR027" H 14100 6000 50  0001 C CNN
+F 1 "+3.3V" H 14100 6290 50  0000 C CNN
+F 2 "" H 14100 6150 50  0000 C CNN
+F 3 "" H 14100 6150 50  0000 C CNN
+	1    14100 6150
 	-1   0    0    1
 $EndComp
@@
 L +3.3V #PWR028
 U 1 1 5A00AB97
-P 12950 6050
-F 0 "#PWR028" H 12950 5900 50  0001 C CNN
-F 1 "+3.3V" H 12950 6190 50  0000 C CNN
-F 2 "" H 12950 6050 50  0000 C CNN
-F 3 "" H 12950 6050 50  0000 C CNN
-	1    12950 6050
+P 12550 6150
+F 0 "#PWR028" H 12550 6000 50  0001 C CNN
+F 1 "+3.3V" H 12550 6290 50  0000 C CNN
+F 2 "" H 12550 6150 50  0000 C CNN
+F 3 "" H 12550 6150 50  0000 C CNN
+	1    12550 6150
 	-1   0    0    1
 $EndComp
@@
 L GND #PWR029
 U 1 1 5A00AC13
-P 13550 4350
-F 0 "#PWR029" H 13550 4100 50  0001 C CNN
-F 1 "GND" H 13550 4200 50  0000 C CNN
-F 2 "" H 13550 4350 50  0000 C CNN
-F 3 "" H 13550 4350 50  0000 C CNN
-	1    13550 4350
+P 13150 4450
+F 0 "#PWR029" H 13150 4200 50  0001 C CNN
+F 1 "GND" H 13150 4300 50  0000 C CNN
+F 2 "" H 13150 4450 50  0000 C CNN
+F 3 "" H 13150 4450 50  0000 C CNN
+	1    13150 4450
 	-1   0    0    1
 $EndComp
@@
 L GND #PWR030
 U 1 1 5A00AC51
-P 14900 4350
-F 0 "#PWR030" H 14900 4100 50  0001 C CNN
-F 1 "GND" H 14900 4200 50  0000 C CNN
-F 2 "" H 14900 4350 50  0000 C CNN
-F 3 "" H 14900 4350 50  0000 C CNN
-	1    14900 4350
-	-1   0    0    1
-$EndComp
-Text GLabel 12650 6050 3    60   Input ~ 0
+P 14700 4450
+F 0 "#PWR030" H 14700 4200 50  0001 C CNN
+F 1 "GND" H 14700 4300 50  0000 C CNN
+F 2 "" H 14700 4450 50  0000 C CNN
+F 3 "" H 14700 4450 50  0000 C CNN
+	1    14700 4450
+	-1   0    0    1
+$EndComp
+Text GLabel 12250 6150 3    60   Input ~ 0
 SD0_DAT2
-Text GLabel 12750 6050 3    60   Input ~ 0
+Text GLabel 12350 6150 3    60   Input ~ 0
 SD0_DAT3
-Text GLabel 12850 6050 3    60   Input ~ 0
+Text GLabel 12450 6150 3    60   Input ~ 0
 SD0_CMD
-Text GLabel 13050 6050 3    60   Input ~ 0
-SDO_CLK
-Text GLabel 13250 6050 3    60   Input ~ 0
+Text GLabel 12650 6150 3    60   Input ~ 0
+SD0_CLK
+Text GLabel 12850 6150 3    60   Input ~ 0
 SD0_DAT0
-Text GLabel 13350 6050 3    60   Input ~ 0
+Text GLabel 12950 6150 3    60   Input ~ 0
 SD0_DAT1
 $Comp
@@
 Text GLabel 14100 3450 3    60   Input ~ 0
 SD1_DAT0
-Text GLabel 14000 6050 3    60   Input ~ 0
+Text GLabel 13800 6150 3    60   Input ~ 0
 SD1_DAT2
-Text GLabel 14100 6050 3    60   Input ~ 0
+Text GLabel 13900 6150 3    60   Input ~ 0
 SD1_DAT3
-Text GLabel 14200 6050 3    60   Input ~ 0
+Text GLabel 14000 6150 3    60   Input ~ 0
 SD1_CMD
-Text GLabel 14400 6050 3    60   Input ~ 0
+Text GLabel 14200 6150 3    60   Input ~ 0
 SD1_CLK
-Text GLabel 14700 6050 3    60   Input ~ 0
+Text GLabel 14500 6150 3    60   Input ~ 0
 SD1_DAT1
-Text GLabel 14600 6050 3    60   Input ~ 0
+Text GLabel 14400 6150 3    60   Input ~ 0
 SD1_DAT0
 Text GLabel 8850 8650 3    60   Input ~ 0
@@
 	0    1    1    0
 $EndComp
-$Comp
-L GND #PWR067
-U 1 1 5A00EB9D
-P 3350 7550
-F 0 "#PWR067" H 3350 7300 50  0001 C CNN
-F 1 "GND" H 3350 7400 50  0000 C CNN
-F 2 "" H 3350 7550 50  0000 C CNN
-F 3 "" H 3350 7550 50  0000 C CNN
-	1    3350 7550
-	0    -1   -1   0
-$EndComp
 Wire Wire Line
 	4500 2050 4300 2050
@@
 	2900 7950 3350 7950
 $Comp
-L GND #PWR068
-U 1 1 5A01EEEA
-P 3350 7950
-F 0 "#PWR068" H 3350 7700 50  0001 C CNN
-F 1 "GND" H 3350 7800 50  0000 C CNN
-F 2 "" H 3350 7950 50  0000 C CNN
-F 3 "" H 3350 7950 50  0000 C CNN
-	1    3350 7950
-	0    -1   -1   0
-$EndComp
-$Comp
-L GND #PWR069
+L GND #PWR067
 U 1 1 5A01EF88
 P 3350 8150
-F 0 "#PWR069" H 3350 7900 50  0001 C CNN
+F 0 "#PWR067" H 3350 7900 50  0001 C CNN
 F 1 "GND" H 3350 8000 50  0000 C CNN
 F 2 "" H 3350 8150 50  0000 C CNN
@@
 	1    0    0    -1
 $EndComp
+NoConn ~ 6650 8650
+NoConn ~ 6750 8650
+NoConn ~ 6850 8650
+NoConn ~ 7150 8650
+NoConn ~ 7650 8650
+NoConn ~ 7750 8650
+NoConn ~ 7850 8650
+NoConn ~ 8050 8650
+NoConn ~ 8150 8650
+NoConn ~ 8250 8650
+NoConn ~ 8350 8650
+NoConn ~ 10050 5350
+NoConn ~ 10050 5250
+NoConn ~ 8950 3950
+NoConn ~ 8850 3950
+NoConn ~ 7850 3950
+NoConn ~ 7750 3950
+NoConn ~ 7650 3950
+NoConn ~ 7550 3950
+NoConn ~ 7350 3950
+NoConn ~ 7250 3950
+NoConn ~ 7150 3950
+NoConn ~ 7050 3950
+NoConn ~ 6850 3950
+NoConn ~ 6750 3950
+NoConn ~ 5350 5450
+NoConn ~ 5350 5550
+NoConn ~ 8500 2050
+NoConn ~ 8400 2050
+NoConn ~ 8300 2050
+NoConn ~ 8200 2050
+NoConn ~ 7500 2050
+NoConn ~ 7400 2050
+NoConn ~ 9200 10300
+$Comp
+L BAT BAT1
+U 1 1 5A040967
+P 7500 10050
+F 0 "BAT1" H 7600 10150 50  0000 L CNN
+F 1 "BAT" H 7600 10050 50  0000 L CNN
+F 2 "" V 7500 10110 50  0000 C CNN
+F 3 "" V 7500 10110 50  0000 C CNN
+	1    7500 10050
+	1    0    0    -1
+$EndComp
+Wire Wire Line
+	3350 7550 3350 8150
+Connection ~ 3350 7950
+$Comp
+L GND #PWR068
+U 1 1 5A0453FE
+P 11100 1750
+F 0 "#PWR068" H 11100 1500 50  0001 C CNN
+F 1 "GND" H 11100 1600 50  0000 C CNN
+F 2 "" H 11100 1750 50  0000 C CNN
+F 3 "" H 11100 1750 50  0000 C CNN
+	1    11100 1750
+	1    0    0    -1
+$EndComp
+$Comp
+L GND #PWR069
+U 1 1 5A045AC1
+P 7550 10150
+F 0 "#PWR069" H 7550 9900 50  0001 C CNN
+F 1 "GND" H 7550 10000 50  0000 C CNN
+F 2 "" H 7550 10150 50  0000 C CNN
+F 3 "" H 7550 10150 50  0000 C CNN
+	1    7550 10150
+	1    0    0    -1
+$EndComp
+$Comp
+L MicroSD CON1
+U 1 1 5A046BC2
+P 12550 5250
+F 0 "CON1" H 11900 5850 50  0000 C CNN
+F 1 "MicroSD" H 13200 5850 50  0000 R CNN
+F 2 "" H 13700 5550 50  0000 C CNN
+F 3 "" H 12550 5250 50  0000 C CNN
+	1    12550 5250
+	0    -1   -1   0
+$EndComp
+$Comp
+L MicroSD CON2
+U 1 1 5A046D0A
+P 14100 5250
+F 0 "CON2" H 13450 5850 50  0000 C CNN
+F 1 "MicroSD" H 14750 5850 50  0000 R CNN
+F 2 "" H 15250 5550 50  0000 C CNN
+F 3 "" H 14100 5250 50  0000 C CNN
+	1    14100 5250
+	0    -1   -1   0
+$EndComp
+Text GLabel 13150 6200 3    60   Input ~ 0
+SD0_CD
+Text GLabel 14700 6200 3    60   Input ~ 0
+SD1_CD
+Text GLabel 7950 3950 1    60   Input ~ 0
+SD1_CD
 $EndSCHEMATC

Commit message: 20171112
Parts:
- added J1: JACK_TRS_6PINS, symbol JACK_TRS_6PINS
- added R4: 100K, symbol R
Connections:
- net +3V3: now also R4.1; no longer U2.5 (MUTE)
- net GND: now also J1.1 (S), J1.4 (SN); no longer P1.3 (P3)
- net INL: now also P1.4 (P4); no longer P1.5 (P5)
- net INR: now also P1.3 (P3); no longer P1.4 (P4)
- net OUTL: now also J1.5 (TN)
- net OUTR: now also J1.6 (RN)
- new net MUTE: J1.2 (T), R4.2, U2.5 (MUTE)
- no-connect marks 34 -> 36
Other:
- note added: "20171112"
- note removed: "20171109"
- moved on the sheet: LS1, LS2
Changed lines of the file:
@@
 handmade01
 Text Notes 13000 11050 0    60   ~ 12
-20171109
+20171112
 $Comp
 L +5V #PWR05
@@
 Text GLabel 1200 5550 3    60   Input ~ 0
 OUTR
-Text GLabel 2200 5500 1    60   Input ~ 0
-OUTL
-Text GLabel 2350 5500 1    60   Input ~ 0
-OUTR
 $Comp
 L C C7
@@
 	0    -1   -1   0
 $EndComp
-$Comp
-L GND #PWR062
-U 1 1 5A00C236
-P 1250 6650
-F 0 "#PWR062" H 1250 6400 50  0001 C CNN
-F 1 "GND" H 1250 6500 50  0000 C CNN
-F 2 "" H 1250 6650 50  0000 C CNN
-F 3 "" H 1250 6650 50  0000 C CNN
-	1    1250 6650
-	1    0    0    -1
-$EndComp
 Text GLabel 1050 6650 3    60   Input ~ 0
 OUTL
 Text GLabel 1150 6650 3    60   Input ~ 0
 OUTR
+Text GLabel 1250 6650 3    60   Input ~ 0
+INR
 Text GLabel 1350 6650 3    60   Input ~ 0
-INR
-Text GLabel 1450 6650 3    60   Input ~ 0
 INL
-Text GLabel 2650 6150 0    60   Input ~ 0
+Text GLabel 3800 9450 0    60   Input ~ 0
 OUT_R+
-Text GLabel 2650 6250 0    60   Input ~ 0
+Text GLabel 3800 9550 0    60   Input ~ 0
 OUT_R-
-Text GLabel 2650 6800 0    60   Input ~ 0
+Text GLabel 3800 10100 0    60   Input ~ 0
 OUT_L+
-Text GLabel 2650 6900 0    60   Input ~ 0
+Text GLabel 3800 10200 0    60   Input ~ 0
 OUT_L-
 Text GLabel 1550 7450 0    60   Input ~ 0
@@
 OUT_L-
 $Comp
-L GND #PWR063
+L GND #PWR062
 U 1 1 5A00E230
 P 1100 7550
-F 0 "#PWR063" H 1100 7300 50  0001 C CNN
+F 0 "#PWR062" H 1100 7300 50  0001 C CNN
 F 1 "GND" H 1100 7400 50  0000 C CNN
 F 2 "" H 1100 7550 50  0000 C CNN
@@
 $EndComp
 $Comp
-L +3.3V #PWR064
+L +3.3V #PWR063
 U 1 1 5A00E3ED
-P 1550 7850
-F 0 "#PWR064" H 1550 7700 50  0001 C CNN
-F 1 "+3.3V" H 1550 7990 50  0000 C CNN
-F 2 "" H 1550 7850 50  0000 C CNN
-F 3 "" H 1550 7850 50  0000 C CNN
-	1    1550 7850
+P 1100 7750
+F 0 "#PWR063" H 1100 7600 50  0001 C CNN
+F 1 "+3.3V" H 1100 7890 50  0000 C CNN
+F 2 "" H 1100 7750 50  0000 C CNN
+F 3 "" H 1100 7750 50  0000 C CNN
+	1    1100 7750
 	0    -1   -1   0
 $EndComp
@@
 $EndComp
 $Comp
-L GND #PWR065
+L GND #PWR064
 U 1 1 5A00E7FD
 P 1550 8450
-F 0 "#PWR065" H 1550 8200 50  0001 C CNN
+F 0 "#PWR064" H 1550 8200 50  0001 C CNN
 F 1 "GND" H 1550 8300 50  0000 C CNN
 F 2 "" H 1550 8450 50  0000 C CNN
@@
 $EndComp
 $Comp
-L +3.3V #PWR066
+L +3.3V #PWR065
 U 1 1 5A00EA61
 P 2900 7850
-F 0 "#PWR066" H 2900 7700 50  0001 C CNN
+F 0 "#PWR065" H 2900 7700 50  0001 C CNN
 F 1 "+3.3V" H 2900 7990 50  0000 C CNN
 F 2 "" H 2900 7850 50  0000 C CNN
@@
 	1000 5400 800  5400
 Wire Wire Line
-	1550 7750 1550 7950
-Connection ~ 1550 7850
-Wire Wire Line
 	2900 7750 2900 7850
 Connection ~ 2900 7850
@@
 	2900 7950 3350 7950
 $Comp
-L GND #PWR067
+L GND #PWR066
 U 1 1 5A01EF88
 P 3350 8150
-F 0 "#PWR067" H 3350 7900 50  0001 C CNN
+F 0 "#PWR066" H 3350 7900 50  0001 C CNN
 F 1 "GND" H 3350 8000 50  0000 C CNN
 F 2 "" H 3350 8150 50  0000 C CNN
 F 3 "" H 3350 8150 50  0000 C CNN
 	1    3350 8150
-	0    -1   -1   0
+	1    0    0    -1
 $EndComp
 Wire Wire Line
@@
 L Speaker LS2
 U 1 1 5A01F987
-P 2850 6800
-F 0 "LS2" H 2900 7025 50  0000 R CNN
-F 1 "SPEAKER_L" H 2900 6950 50  0000 R CNN
-F 2 "" H 2850 6600 50  0000 C CNN
-F 3 "" H 2840 6750 50  0000 C CNN
-	1    2850 6800
+P 4000 10100
+F 0 "LS2" H 4050 10325 50  0000 R CNN
+F 1 "SPEAKER_L" H 4050 10250 50  0000 R CNN
+F 2 "" H 4000 9900 50  0000 C CNN
+F 3 "" H 3990 10050 50  0000 C CNN
+	1    4000 10100
 	1    0    0    -1
 $EndComp
@@
 L Speaker LS1
 U 1 1 5A01FA5B
-P 2850 6150
-F 0 "LS1" H 2900 6375 50  0000 R CNN
-F 1 "SPEAKER_R" H 2900 6300 50  0000 R CNN
-F 2 "" H 2850 5950 50  0000 C CNN
-F 3 "" H 2840 6100 50  0000 C CNN
-	1    2850 6150
+P 4000 9450
+F 0 "LS1" H 4050 9675 50  0000 R CNN
+F 1 "SPEAKER_R" H 4050 9600 50  0000 R CNN
+F 2 "" H 4000 9250 50  0000 C CNN
+F 3 "" H 3990 9400 50  0000 C CNN
+	1    4000 9450
 	1    0    0    -1
 $EndComp
@@
 Connection ~ 3350 7950
 $Comp
-L GND #PWR068
+L GND #PWR067
 U 1 1 5A0453FE
 P 11100 1750
-F 0 "#PWR068" H 11100 1500 50  0001 C CNN
+F 0 "#PWR067" H 11100 1500 50  0001 C CNN
 F 1 "GND" H 11100 1600 50  0000 C CNN
 F 2 "" H 11100 1750 50  0000 C CNN
@@
 $EndComp
 $Comp
-L GND #PWR069
+L GND #PWR068
 U 1 1 5A045AC1
 P 7550 10150
-F 0 "#PWR069" H 7550 9900 50  0001 C CNN
+F 0 "#PWR068" H 7550 9900 50  0001 C CNN
 F 1 "GND" H 7550 10000 50  0000 C CNN
 F 2 "" H 7550 10150 50  0000 C CNN
@@
 Text GLabel 7950 3950 1    60   Input ~ 0
 SD1_CD
+Wire Wire Line
+	1100 7750 1550 7750
+Connection ~ 1100 7750
+Text GLabel 1550 7850 0    60   Input ~ 0
+MUTE
+Wire Wire Line
+	1550 7950 1100 7950
+Wire Wire Line
+	1100 7950 1100 7750
+$Comp
+L JACK_TRS_6PINS J1
+U 1 1 5A07D9F4
+P 1800 9800
+F 0 "J1" H 1800 10200 50  0000 C CNN
+F 1 "JACK_TRS_6PINS" H 1750 9500 50  0000 C CNN
+F 2 "" H 1900 9650 50  0000 C CNN
+F 3 "" H 1900 9650 50  0000 C CNN
+	1    1800 9800
+	1    0    0    -1
+$EndComp
+$Comp
+L GND #PWR069
+U 1 1 5A07DB46
+P 2200 9500
+F 0 "#PWR069" H 2200 9250 50  0001 C CNN
+F 1 "GND" H 2200 9350 50  0000 C CNN
+F 2 "" H 2200 9500 50  0000 C CNN
+F 3 "" H 2200 9500 50  0000 C CNN
+	1    2200 9500
+	0    -1   -1   0
+$EndComp
+Wire Wire Line
+	2200 9600 2200 9500
+Connection ~ 2200 9500
+Text GLabel 2200 9700 2    60   Input ~ 0
+OUTL
+Text GLabel 2200 9900 2    60   Input ~ 0
+OUTR
+$Comp
+L R R4
+U 1 1 5A08601E
+P 2850 9650
+F 0 "R4" V 2930 9650 50  0000 C CNN
+F 1 "100K" V 2850 9650 50  0000 C CNN
+F 2 "" V 2780 9650 50  0000 C CNN
+F 3 "" H 2850 9650 50  0000 C CNN
+	1    2850 9650
+	1    0    0    -1
+$EndComp
+$Comp
+L +3.3V #PWR070
+U 1 1 5A0860D1
+P 2850 9500
+F 0 "#PWR070" H 2850 9350 50  0001 C CNN
+F 1 "+3.3V" H 2850 9640 50  0000 C CNN
+F 2 "" H 2850 9500 50  0000 C CNN
+F 3 "" H 2850 9500 50  0000 C CNN
+	1    2850 9500
+	1    0    0    -1
+$EndComp
+Wire Wire Line
+	2200 9800 2850 9800
+Text GLabel 2850 9800 3    60   Input ~ 0
+MUTE
+Connection ~ 2850 9800
+NoConn ~ 2200 10000
+NoConn ~ 1450 6650
 $EndSCHEMATC

Commit message: 20171115
Connections:
- net +3V3: no longer U2.12 (SHND)
- net MUTE: now also U2.12 (SHND)
Other:
- note added: "20171115"
- note removed: "20171112"
Changed lines of the file:
@@
 handmade01
 Text Notes 13000 11050 0    60   ~ 12
-20171112
+20171115
 $Comp
 L +5V #PWR05
@@
 L +3.3V #PWR065
 U 1 1 5A00EA61
-P 2900 7850
-F 0 "#PWR065" H 2900 7700 50  0001 C CNN
-F 1 "+3.3V" H 2900 7990 50  0000 C CNN
-F 2 "" H 2900 7850 50  0000 C CNN
-F 3 "" H 2900 7850 50  0000 C CNN
-	1    2900 7850
+P 2900 7750
+F 0 "#PWR065" H 2900 7600 50  0001 C CNN
+F 1 "+3.3V" H 2900 7890 50  0000 C CNN
+F 2 "" H 2900 7750 50  0000 C CNN
+F 3 "" H 2900 7750 50  0000 C CNN
+	1    2900 7750
 	0    1    1    0
 $EndComp
@@
 Wire Wire Line
 	1000 5400 800  5400
-Wire Wire Line
-	2900 7750 2900 7850
-Connection ~ 2900 7850
 Wire Wire Line
 	2900 7950 3350 7950
@@
 NoConn ~ 2200 10000
 NoConn ~ 1450 6650
+Text GLabel 2900 7850 2    60   Input ~ 0
+MUTE
 $EndSCHEMATC

Commit message: 20171121
Parts:
- BAT1, P6: footprint (none) -> Connectors_Molex:Molex_SPOX-5267_22-03-5035_03x2.54mm_Straight
- C1, C10, C11, C12, C2, C3, C4, C5, C6, C7, C8, C9: footprint (none) -> Capacitors_SMD:C_0603_HandSoldering
- CON1, CON2: footprint (none) -> Connectors:microSD_Card_Receptacle_Wuerth_693072010801
- J1: footprint (none) -> Connectors:PJ311_3.5mm_Jack
- LS1, LS2: footprint (none) -> Resistors_SMD:R_2010_HandSoldering
- P1: footprint (none) -> mylib:volumn
- P4: footprint (none) -> Connectors:USB_Micro-B
- Q1: footprint (none) -> TO_SOT_Packages_SMD:SOT-23-5_HandSoldering
- R1, R2, R3, R4: footprint (none) -> Resistors_SMD:R_0603_HandSoldering
- RN1, RN2: footprint Resistors_ThroughHole:Resistor_Array_SIP7 -> Connectors_Molex:Molex_KK-6410-07_07x2.54mm_Straight
- RN3: footprint Resistors_ThroughHole:Resistor_Array_SIP13 -> Connectors_Molex:Molex_KK-6410-13_13x2.54mm_Straight
- SW1, SW10, SW9: footprint (none) -> Buttons_Switches_THT:SW_Tactile_SKHH_Angled
- SW11, SW14, SW5, SW6: footprint (none) -> mylib:dpad-h
- SW12, SW13, SW3, SW4: footprint (none) -> mylib:dpad-v
- SW2: footprint (none) -> Buttons_Switches_THT:SW_Tactile_SPST_Angled_PTS645Vx31-2LFS
- SW7, SW8: footprint (none) -> Buttons_Switches_SMD:SW_SPST_SKQG
- U1: footprint (none) -> Housings_SSOP:TSSOP-20_4.4x6.5mm_Pitch0.65mm
- U2: footprint (none) -> Housings_SSOP:SOP-16_4.4x10.4mm_Pitch1.27mm
- U3: footprint (none) -> mylib:fpc-45pin-0.5mm
- U4: footprint (none) -> mylib:cm3354
- U5: footprint (none) -> Housings_SOIC:SO-5_4.4x3.6mm_Pitch1.27mm
Other:
- note added: "20171121"
- note removed: "20171115"

Commit message: 20171129
Parts:
- removed RN1: SD0_4.7K, Connectors_Molex:Molex_KK-6410-07_07x2.54mm_Straight, symbol R_Network06
- removed RN2: SD1_4.7K, Connectors_Molex:Molex_KK-6410-07_07x2.54mm_Straight, symbol R_Network06
- removed RN3: GAMEPAD_4.7K, Connectors_Molex:Molex_KK-6410-13_13x2.54mm_Straight, symbol R_Network12
- added R10, R11, R12, R13, R14, R15, R16, R17, R18, R19, R20, R21, R22, R23, R24, R25, R26, R27, R28, R5, R6, R7, R8, R9: 4.7K, Resistors_SMD:R_0603_HandSoldering, symbol R
Connections:
- net +3V3: now also R10.1, R11.1, R12.1, R13.1, R14.1, R15.1, R16.1, R17.1, R18.1, R19.1, R20.1, R21.1, R22.1, R23.1, R24.1, R25.1, R26.1, R27.1, R28.1, R5.1, R6.1, R7.1, R8.1, R9.1
- net A: now also R24.2
- net B: now also R26.2
- net DOWN: now also R12.2
- net L: now also R20.2
- net LEFT: now also R13.2
- net R: now also R22.2
- net RIGHT: now also R14.2
- net SD0_CD: now also CON1.10 (INSERT)
- net SD0_CLK: now also R7.2
- net SD0_CMD: now also R8.2
- net SD0_DAT0: now also R11.2
- net SD0_DAT1: now also R9.2
- net SD0_DAT2: now also R6.2
- net SD0_DAT3: now also R5.2
- net SD1_CD: now also CON2.10 (INSERT)
- net SD1_CLK: now also R19.2
- net SD1_CMD: now also R21.2
- net SD1_DAT0: now also R25.2
- net SD1_DAT1: now also R23.2
- net SD1_DAT2: now also R17.2
- net SD1_DAT3: now also R15.2
- net SELECT: now also R16.2
- net START: now also R18.2
- net UP: now also R10.2
- net X: now also R27.2
- net Y: now also R28.2
Other:
- note added: "20171129"
- note removed: "20171121"
