File: handmade01/main.sch (KiCad schematic (older format))
At the start: 69 parts, among them CON1 MicroSD, CON2 MicroSD, J1 JACK_TRS_6PINS, P1 VOLUMN, P4 USB_OTG, P6 UART_DEBUG, Q1 1AM, SW1 POWER, SW10 R, SW11 A, SW12 B, SW13 X, SW14 Y, SW2 RESET, SW3 UP, SW4 DOWN, SW5 LEFT, SW6 RIGHT, SW7 SELECT, SW8 START, SW9 L, U1 PCM5102A, U2 PAM8403, U3 IPS_2.4_240x320_ST7789V, U4 CM3354, U5 TPS71718

Commit message: 20171130
Parts:
- removed SW1: POWER, Buttons_Switches_THT:SW_Tactile_SKHH_Angled, symbol SW_Push_Dual_x2
- removed SW10: R, Buttons_Switches_THT:SW_Tactile_SKHH_Angled, symbol SW_Push_Dual_x2
- removed SW11: A, mylib:dpad-h, symbol SW_Push_Dual_x2
- removed SW12: B, mylib:dpad-v, symbol SW_Push_Dual_x2
- removed SW13: X, mylib:dpad-v, symbol SW_Push_Dual_x2
- removed SW14: Y, mylib:dpad-h, symbol SW_Push_Dual_x2
- removed SW2: RESET, Buttons_Switches_THT:SW_Tactile_SPST_Angled_PTS645Vx31-2LFS, symbol SW_Push_Dual_x2
- removed SW3: UP, mylib:dpad-v, symbol SW_Push_Dual_x2
- removed SW4: DOWN, mylib:dpad-v, symbol SW_Push_Dual_x2
- removed SW5: LEFT, mylib:dpad-h, symbol SW_Push_Dual_x2
- removed SW6: RIGHT, mylib:dpad-h, symbol SW_Push_Dual_x2
- removed SW7: SELECT, Buttons_Switches_SMD:SW_SPST_SKQG, symbol SW_Push_Dual_x2
- removed SW8: START, Buttons_Switches_SMD:SW_SPST_SKQG, symbol SW_Push_Dual_x2
- removed SW9: L, Buttons_Switches_THT:SW_Tactile_SKHH_Angled, symbol SW_Push_Dual_x2
- added SW1: POWER, Buttons_Switches_THT:SW_PUSH_6mm, symbol SW_Push
- added SW10: R, Buttons_Switches_THT:SW_PUSH_6mm, symbol SW_Push
- added SW11: A, mylib:dpad-h, symbol SW_Push
- added SW12: B, mylib:dpad-v, symbol SW_Push
- added SW13: X, mylib:dpad-h, symbol SW_Push
- added SW14: Y, mylib:dpad-v, symbol SW_Push
- added SW2: Reset, Buttons_Switches_THT:SW_PUSH_6mm, symbol SW_Push
- added SW3: UP, mylib:dpad-v, symbol SW_Push
- added SW4: Down, mylib:dpad-v, symbol SW_Push
- added SW5: Left, mylib:dpad-h, symbol SW_Push
- added SW6: Right, mylib:dpad-h, symbol SW_Push
- added SW7: Select, Buttons_Switches_SMD:SW_SPST_TL3342, symbol SW_Push
- added SW8: Start, Buttons_Switches_SMD:SW_SPST_TL3342, symbol SW_Push
- added SW9: L, Buttons_Switches_THT:SW_PUSH_6mm, symbol SW_Push
- CON1, CON2: footprint Connectors:microSD_Card_Receptacle_Wuerth_693072010801 -> mylib:microsd
- U5: footprint Housings_SOIC:SO-5_4.4x3.6mm_Pitch1.27mm -> mylib:sc-70-5
Other:
- note added: "20171130"
- note removed: "20171129"
Changed lines of the file:
@@
 handmade01
 Text Notes 13000 11050 0    60   ~ 12
-20171129
+20171130
 $Comp
 L +5V #PWR05
@@
 F 0 "U5" H 8650 10500 60  0000 C CNN
 F 1 "TPS71718" H 8800 10400 60  0000 C CNN
-F 2 "Housings_SOIC:SO-5_4.4x3.6mm_Pitch1.27mm" H 8850 10400 60  0000 C CNN
+F 2 "mylib:sc-70-5" H 8850 10400 60  0000 C CNN
 F 3 "" H 8850 10400 60  0000 C CNN
 	1    8850 10200
@@
 	1    9200 9800
 	-1   0    0    1
-$EndComp
-$Comp
-L SW_Push_Dual_x2 SW1
-U 1 1 59FFF5DC
-P 11800 9200
-F 0 "SW1" H 11850 9300 50  0000 L CNN
-F 1 "POWER" H 11800 9140 50  0000 C CNN
-F 2 "Buttons_Switches_THT:SW_Tactile_SKHH_Angled" H 11800 9400 50  0000 C CNN
-F 3 "" H 11800 9400 50  0000 C CNN
-	1    11800 9200
-	0    1    1    0
-$EndComp
-$Comp
-L SW_Push_Dual_x2 SW2
-U 1 1 59FFF626
-P 12050 9200
-F 0 "SW2" H 12100 9300 50  0000 L CNN
-F 1 "RESET" H 12050 9140 50  0000 C CNN
-F 2 "Buttons_Switches_THT:SW_Tactile_SPST_Angled_PTS645Vx31-2LFS" H 12050 9400 50  0000 C CNN
-F 3 "" H 12050 9400 50  0000 C CNN
-	1    12050 9200
-	0    1    1    0
 $EndComp
 $Comp
@@
 SD1_DAT3
 $Comp
-L SW_Push_Dual_x2 SW3
-U 1 1 5A00E313
-P 12300 9200
-F 0 "SW3" H 12350 9300 50  0000 L CNN
-F 1 "UP" H 12300 9140 50  0000 C CNN
-F 2 "mylib:dpad-v" H 12300 9400 50  0000 C CNN
-F 3 "" H 12300 9400 50  0000 C CNN
-	1    12300 9200
-	0    1    1    0
-$EndComp
-$Comp
-L SW_Push_Dual_x2 SW4
-U 1 1 5A00E319
-P 12550 9200
-F 0 "SW4" H 12600 9300 50  0000 L CNN
-F 1 "DOWN" H 12550 9140 50  0000 C CNN
-F 2 "mylib:dpad-v" H 12550 9400 50  0000 C CNN
-F 3 "" H 12550 9400 50  0000 C CNN
-	1    12550 9200
-	0    1    1    0
-$EndComp
-$Comp
 L GND #PWR031
 U 1 1 5A00E31F
@@
 $EndComp
 $Comp
-L SW_Push_Dual_x2 SW5
-U 1 1 5A00E455
-P 12800 9200
-F 0 "SW5" H 12850 9300 50  0000 L CNN
-F 1 "LEFT" H 12800 9140 50  0000 C CNN
-F 2 "mylib:dpad-h" H 12800 9400 50  0000 C CNN
-F 3 "" H 12800 9400 50  0000 C CNN
-	1    12800 9200
-	0    1    1    0
-$EndComp
-$Comp
-L SW_Push_Dual_x2 SW6
-U 1 1 5A00E45B
-P 13050 9200
-F 0 "SW6" H 13100 9300 50  0000 L CNN
-F 1 "RIGHT" H 13050 9140 50  0000 C CNN
-F 2 "mylib:dpad-h" H 13050 9400 50  0000 C CNN
-F 3 "" H 13050 9400 50  0000 C CNN
-	1    13050 9200
-	0    1    1    0
-$EndComp
-$Comp
 L GND #PWR033
 U 1 1 5A00E461
@@
 $EndComp
 $Comp
-L SW_Push_Dual_x2 SW7
-U 1 1 5A00E46D
-P 13300 9200
-F 0 "SW7" H 13350 9300 50  0000 L CNN
-F 1 "SELECT" H 13300 9140 50  0000 C CNN
-F 2 "Buttons_Switches_SMD:SW_SPST_SKQG" H 13300 9400 50  0000 C CNN
-F 3 "" H 13300 9400 50  0000 C CNN
-	1    13300 9200
-	0    1    1    0
-$EndComp
-$Comp
-L SW_Push_Dual_x2 SW8
-U 1 1 5A00E473
-P 13550 9200
-F 0 "SW8" H 13600 9300 50  0000 L CNN
-F 1 "START" H 13550 9140 50  0000 C CNN
-F 2 "Buttons_Switches_SMD:SW_SPST_SKQG" H 13550 9400 50  0000 C CNN
-F 3 "" H 13550 9400 50  0000 C CNN
-	1    13550 9200
-	0    1    1    0
-$EndComp
-$Comp
 L GND #PWR035
 U 1 1 5A00E479
@@
 $EndComp
 $Comp
-L SW_Push_Dual_x2 SW9
-U 1 1 5A00E67B
-P 13800 9200
-F 0 "SW9" H 13850 9300 50  0000 L CNN
-F 1 "L" H 13800 9140 50  0000 C CNN
-F 2 "Buttons_Switches_THT:SW_Tactile_SKHH_Angled" H 13800 9400 50  0000 C CNN
-F 3 "" H 13800 9400 50  0000 C CNN
-	1    13800 9200
-	0    1    1    0
-$EndComp
-$Comp
-L SW_Push_Dual_x2 SW10
-U 1 1 5A00E681
-P 14050 9200
-F 0 "SW10" H 14100 9300 50  0000 L CNN
-F 1 "R" H 14050 9140 50  0000 C CNN
-F 2 "Buttons_Switches_THT:SW_Tactile_SKHH_Angled" H 14050 9400 50  0000 C CNN
-F 3 "" H 14050 9400 50  0000 C CNN
-	1    14050 9200
-	0    1    1    0
-$EndComp
-$Comp
 L GND #PWR037
 U 1 1 5A00E687
@@
 $EndComp
 $Comp
-L SW_Push_Dual_x2 SW11
-U 1 1 5A00E693
-P 14300 9200
-F 0 "SW11" H 14350 9300 50  0000 L CNN
-F 1 "A" H 14300 9140 50  0000 C CNN
-F 2 "mylib:dpad-h" H 14300 9400 50  0000 C CNN
-F 3 "" H 14300 9400 50  0000 C CNN
-	1    14300 9200
-	0    1    1    0
-$EndComp
-$Comp
-L SW_Push_Dual_x2 SW12
-U 1 1 5A00E699
-P 14550 9200
-F 0 "SW12" H 14600 9300 50  0000 L CNN
-F 1 "B" H 14550 9140 50  0000 C CNN
-F 2 "mylib:dpad-v" H 14550 9400 50  0000 C CNN
-F 3 "" H 14550 9400 50  0000 C CNN
-	1    14550 9200
-	0    1    1    0
-$EndComp
-$Comp
 L GND #PWR039
 U 1 1 5A00E69F
@@
 	1    14550 9400
 	1    0    0    -1
-$EndComp
-$Comp
-L SW_Push_Dual_x2 SW13
-U 1 1 5A00E6AB
-P 14800 9200
-F 0 "SW13" H 14850 9300 50  0000 L CNN
-F 1 "X" H 14800 9140 50  0000 C CNN
-F 2 "mylib:dpad-v" H 14800 9400 50  0000 C CNN
-F 3 "" H 14800 9400 50  0000 C CNN
-	1    14800 9200
-	0    1    1    0
-$EndComp
-$Comp
-L SW_Push_Dual_x2 SW14
-U 1 1 5A00E6B1
-P 15050 9200
-F 0 "SW14" H 15100 9300 50  0000 L CNN
-F 1 "Y" H 15050 9140 50  0000 C CNN
-F 2 "mylib:dpad-h" H 15050 9400 50  0000 C CNN
-F 3 "" H 15050 9400 50  0000 C CNN
-	1    15050 9200
-	0    1    1    0
 $EndComp
 $Comp
@@
 F 0 "CON1" H 11900 5850 50  0000 C CNN
 F 1 "MicroSD" H 13200 5850 50  0000 R CNN
-F 2 "Connectors:microSD_Card_Receptacle_Wuerth_693072010801" H 13700 5550 50  0000 C CNN
+F 2 "mylib:microsd" H 13700 5550 50  0000 C CNN
 F 3 "" H 12550 5250 50  0000 C CNN
 	1    12550 5250
@@
 F 0 "CON2" H 13450 5850 50  0000 C CNN
 F 1 "MicroSD" H 14750 5850 50  0000 R CNN
-F 2 "Connectors:microSD_Card_Receptacle_Wuerth_693072010801" H 15250 5550 50  0000 C CNN
+F 2 "mylib:microsd" H 15250 5550 50  0000 C CNN
 F 3 "" H 14100 5250 50  0000 C CNN
 	1    14100 5250
@@
 Connection ~ 13850 7250
 Connection ~ 13950 7250
+$Comp
+L SW_Push SW1
+U 1 1 5A1FE007
+P 11800 9200
+F 0 "SW1" H 11850 9300 50  0000 L CNN
+F 1 "POWER" H 11800 9140 50  0000 C CNN
+F 2 "Buttons_Switches_THT:SW_PUSH_6mm" H 11800 9400 50  0001 C CNN
+F 3 "" H 11800 9400 50  0001 C CNN
+	1    11800 9200
+	0    1    1    0
+$EndComp
+$Comp
+L SW_Push SW2
+U 1 1 5A20183B
+P 12050 9200
+F 0 "SW2" H 12100 9300 50  0000 L CNN
+F 1 "Reset" H 12050 9140 50  0000 C CNN
+F 2 "Buttons_Switches_THT:SW_PUSH_6mm" H 12050 9400 50  0001 C CNN
+F 3 "" H 12050 9400 50  0001 C CNN
+	1    12050 9200
+	0    1    1    0
+$EndComp
+$Comp
+L SW_Push SW3
+U 1 1 5A201A49
+P 12300 9200
+F 0 "SW3" H 12350 9300 50  0000 L CNN
+F 1 "UP" H 12300 9140 50  0000 C CNN
+F 2 "mylib:dpad-v" H 12300 9400 50  0001 C CNN
+F 3 "" H 12300 9400 50  0001 C CNN
+	1    12300 9200
+	0    1    1    0
+$EndComp
+$Comp
+L SW_Push SW4
+U 1 1 5A201F18
+P 12550 9250
+F 0 "SW4" H 12600 9350 50  0000 L CNN
+F 1 "Down" H 12550 9190 50  0000 C CNN
+F 2 "mylib:dpad-v" H 12550 9450 50  0001 C CNN
+F 3 "" H 12550 9450 50  0001 C CNN
+	1    12550 9250
+	0    1    1    0
+$EndComp
+$Comp
+L SW_Push SW5
+U 1 1 5A2026FB
+P 12800 9200
+F 0 "SW5" H 12850 9300 50  0000 L CNN
+F 1 "Left" H 12800 9140 50  0000 C CNN
+F 2 "mylib:dpad-h" H 12800 9400 50  0001 C CNN
+F 3 "" H 12800 9400 50  0001 C CNN
+	1    12800 9200
+	0    1    1    0
+$EndComp
+$Comp
+L SW_Push SW6
+U 1 1 5A202A1C
+P 13050 9200
+F 0 "SW6" H 13100 9300 50  0000 L CNN
+F 1 "Right" H 13050 9140 50  0000 C CNN
+F 2 "mylib:dpad-h" H 13050 9400 50  0001 C CNN
+F 3 "" H 13050 9400 50  0001 C CNN
+	1    13050 9200
+	0    1    1    0
+$EndComp
+$Comp
+L SW_Push SW7
+U 1 1 5A202D3D
+P 13300 9200
+F 0 "SW7" H 13350 9300 50  0000 L CNN
+F 1 "Select" H 13300 9140 50  0000 C CNN
+F 2 "Buttons_Switches_SMD:SW_SPST_TL3342" H 13300 9400 50  0001 C CNN
+F 3 "" H 13300 9400 50  0001 C CNN
+	1    13300 9200
+	0    1    1    0
+$EndComp
+$Comp
+L SW_Push SW8
+U 1 1 5A202F43
+P 13550 9200
+F 0 "SW8" H 13600 9300 50  0000 L CNN
+F 1 "Start" H 13550 9140 50  0000 C CNN
+F 2 "Buttons_Switches_SMD:SW_SPST_TL3342" H 13550 9400 50  0001 C CNN
+F 3 "" H 13550 9400 50  0001 C CNN
+	1    13550 9200
+	0    1    1    0
+$EndComp
+$Comp
+L SW_Push SW9
+U 1 1 5A20321F
+P 13800 9200
+F 0 "SW9" H 13850 9300 50  0000 L CNN
+F 1 "L" H 13800 9140 50  0000 C CNN
+F 2 "Buttons_Switches_THT:SW_PUSH_6mm" H 13800 9400 50  0001 C CNN
+F 3 "" H 13800 9400 50  0001 C CNN
+	1    13800 9200
+	0    1    1    0
+$EndComp
+$Comp
+L SW_Push SW10
+U 1 1 5A2037A6
+P 14050 9200
+F 0 "SW10" H 14100 9300 50  0000 L CNN
+F 1 "R" H 14050 9140 50  0000 C CNN
+F 2 "Buttons_Switches_THT:SW_PUSH_6mm" H 14050 9400 50  0001 C CNN
+F 3 "" H 14050 9400 50  0001 C CNN
+	1    14050 9200
+	0    1    1    0
+$EndComp
+$Comp
+L SW_Push SW11
+U 1 1 5A2039AC
+P 14300 9200
+F 0 "SW11" H 14350 9300 50  0000 L CNN
+F 1 "A" H 14300 9140 50  0000 C CNN
+F 2 "mylib:dpad-h" H 14300 9400 50  0001 C CNN
+F 3 "" H 14300 9400 50  0001 C CNN
+	1    14300 9200
+	0    1    1    0
+$EndComp
+$Comp
+L SW_Push SW12
+U 1 1 5A203D5E
+P 14550 9200
+F 0 "SW12" H 14600 9300 50  0000 L CNN
+F 1 "B" H 14550 9140 50  0000 C CNN
+F 2 "mylib:dpad-v" H 14550 9400 50  0001 C CNN
+F 3 "" H 14550 9400 50  0001 C CNN
+	1    14550 9200
+	0    1    1    0
+$EndComp
+$Comp
+L SW_Push SW13
+U 1 1 5A203FA8
+P 14800 9200
+F 0 "SW13" H 14850 9300 50  0000 L CNN
+F 1 "X" H 14800 9140 50  0000 C CNN
+F 2 "mylib:dpad-h" H 14800 9400 50  0001 C CNN
+F 3 "" H 14800 9400 50  0001 C CNN
+	1    14800 9200
+	0    1    1    0
+$EndComp
+$Comp
+L SW_Push SW14
+U 1 1 5A2041F2
+P 15050 9200
+F 0 "SW14" H 15100 9300 50  0000 L CNN
+F 1 "Y" H 15050 9140 50  0000 C CNN
+F 2 "mylib:dpad-v" H 15050 9400 50  0001 C CNN
+F 3 "" H 15050 9400 50  0001 C CNN
+	1    15050 9200
+	0    1    1    0
+$EndComp
 $EndSCHEMATC

Commit message: 20171130
Parts:
- J1: footprint Connectors:PJ311_3.5mm_Jack -> mylib:pj311_3.5mm
Changed lines of the file:
@@
 F 0 "J1" H 1800 10200 50  0000 C CNN
 F 1 "JACK_TRS_6PINS" H 1750 9500 50  0000 C CNN
-F 2 "Connectors:PJ311_3.5mm_Jack" H 1900 9650 50  0000 C CNN
+F 2 "mylib:pj311_3.5mm" H 1900 9650 50  0000 C CNN
 F 3 "" H 1900 9650 50  0000 C CNN
 	1    1800 9800

Commit message: 20171201
Parts:
- BAT1, P6: footprint Connectors_Molex:Molex_SPOX-5267_22-03-5035_03x2.54mm_Straight -> Connectors:GS3
- LS1, LS2: footprint Resistors_SMD:R_2010_HandSoldering -> Connectors:GS2
- U3: footprint mylib:fpc-45pin-0.5mm -> mylib:fpc-45pin-0.5mm-down
Other:
- note added: "20171201"
- note removed: "20171130"
Changed lines of the file:
@@
 handmade01
 Text Notes 13000 11050 0    60   ~ 12
-20171130
+20171201
 $Comp
 L +5V #PWR05
@@
 F 0 "U3" H 4150 1850 60  0000 C CNN
 F 1 "IPS_2.4_240x320_ST7789V" H 4700 1750 60  0000 C CNN
-F 2 "mylib:fpc-45pin-0.5mm" H 5150 1500 60  0000 C CNN
+F 2 "mylib:fpc-45pin-0.5mm-down" H 5150 1500 60  0000 C CNN
 F 3 "" H 5150 1500 60  0000 C CNN
 	1    5900 1500
@@
 F 0 "P6" H 11200 1750 50  0000 C CNN
 F 1 "UART_DEBUG" V 11300 1550 50  0000 C CNN
-F 2 "Connectors_Molex:Molex_SPOX-5267_22-03-5035_03x2.54mm_Straight" H 11200 1550 50  0000 C CNN
+F 2 "Connectors:GS3" H 11200 1550 50  0000 C CNN
 F 3 "" H 11200 1550 50  0000 C CNN
 	1    11200 1550
@@
 F 0 "LS2" H 4050 10325 50  0000 R CNN
 F 1 "SPEAKER_L" H 4050 10250 50  0000 R CNN
-F 2 "Resistors_SMD:R_2010_HandSoldering" H 4000 9900 50  0000 C CNN
+F 2 "Connectors:GS2" H 4000 9900 50  0000 C CNN
 F 3 "" H 3990 10050 50  0000 C CNN
 	1    4000 10100
@@
 F 0 "LS1" H 4050 9675 50  0000 R CNN
 F 1 "SPEAKER_R" H 4050 9600 50  0000 R CNN
-F 2 "Resistors_SMD:R_2010_HandSoldering" H 4000 9250 50  0000 C CNN
+F 2 "Connectors:GS2" H 4000 9250 50  0000 C CNN
 F 3 "" H 3990 9400 50  0000 C CNN
 	1    4000 9450
@@
 F 0 "BAT1" H 7600 10150 50  0000 L CNN
 F 1 "BAT" H 7600 10050 50  0000 L CNN
-F 2 "Connectors_Molex:Molex_SPOX-5267_22-03-5035_03x2.54mm_Straight" V 7500 10110 50  0000 C CNN
+F 2 "Connectors:GS3" V 7500 10110 50  0000 C CNN
 F 3 "" V 7500 10110 50  0000 C CNN
 	1    7500 10050

Commit message: 20171204
Parts:
- P4: footprint Connectors:USB_Micro-B -> Connectors:USB_Mini-B
Changed lines of the file:
@@
 F 0 "P4" H 6725 9675 50  0000 C CNN
 F 1 "USB_OTG" H 6400 10000 50  0000 C CNN
-F 2 "Connectors:USB_Micro-B" V 6350 9700 50  0000 C CNN
+F 2 "Connectors:USB_Mini-B" V 6350 9700 50  0000 C CNN
 F 3 "" V 6350 9700 50  0000 C CNN
 	1    6400 9800

Commit message: 20171207
Other:
- note added: "Handmade01"
- note removed: "1.0"
- note removed: "20171201"
- note removed: "handmade01"
Changed lines of the file:
@@
 EESchema Schematic File Version 2
-LIBS:main-rescue
 LIBS:power
 LIBS:device
@@
 LIBS:memory
 LIBS:xilinx
+LIBS:special
 LIBS:microcontrollers
 LIBS:dsp
@@
 LIBS:contrib
 LIBS:valves
-LIBS:switches
-LIBS:mysch
 LIBS:main-cache
-EELAYER 25 0
+EELAYER 27 0
 EELAYER END
 $Descr A3 16535 11693
@@
 Sheet 1 1
 Title ""
-Date ""
+Date "7 dec 2017"
 Rev ""
 Comp ""
@@
 Comment4 ""
 $EndDescr
-Text Notes 15420 11060 0    60   ~ 12
-1.0
 $Comp
 L CM3354 U4
@@
 	-1   0    0    1
 $EndComp
-Text Notes 12250 10950 0    98   ~ 20
-handmade01
-Text Notes 13000 11050 0    60   ~ 12
-20171201
 $Comp
 L +5V #PWR05
@@
 	0    1    1    0
 $EndComp
+Text Notes 12175 10975 0    60   ~ 12
+Handmade01
 $EndSCHEMATC

Commit message: 20171207
Parts:
- C10, C9: footprint Capacitors_SMD:C_0603_HandSoldering -> (none)
- U1: footprint Housings_SSOP:TSSOP-20_4.4x6.5mm_Pitch0.65mm -> (none)
Changed lines of the file:
@@
 F 0 "U1" H 2050 5100 60  0000 C CNN
 F 1 "PCM5102A" H 2200 5000 60  0000 C CNN
-F 2 "Housings_SSOP:TSSOP-20_4.4x6.5mm_Pitch0.65mm" H 2200 4800 60  0000 C CNN
+F 2 "" H 2200 4800 60  0000 C CNN
 F 3 "" H 2200 4800 60  0000 C CNN
 	1    2300 4450
@@
 F 0 "C10" H 3625 4200 50  0000 L CNN
 F 1 "0.1uF" H 3625 4000 50  0000 L CNN
-F 2 "Capacitors_SMD:C_0603_HandSoldering" H 3638 3950 50  0000 C CNN
+F 2 "" H 3638 3950 50  0000 C CNN
 F 3 "" H 3600 4100 50  0000 C CNN
 	1    3600 4100
@@
 F 0 "C9" H 2975 3700 50  0000 L CNN
 F 1 "0.1uF" H 2975 3500 50  0000 L CNN
-F 2 "Capacitors_SMD:C_0603_HandSoldering" H 2988 3450 50  0000 C CNN
+F 2 "" H 2988 3450 50  0000 C CNN
 F 3 "" H 2950 3600 50  0000 C CNN
 	1    2950 3600

Commit message: 20171207
Parts:
- BAT1, P6: footprint Connectors:GS3 -> (none)
- C1, C11, C12, C2, C3, C4, C5, C6, C7, C8: footprint Capacitors_SMD:C_0603_HandSoldering -> (none)
- CON1, CON2: footprint mylib:microsd -> (none)
- J1: footprint mylib:pj311_3.5mm -> (none)
- LS1, LS2: footprint Connectors:GS2 -> (none)
- P1: footprint mylib:volumn -> (none)
- P4: footprint Connectors:USB_Mini-B -> (none)
- Q1: footprint TO_SOT_Packages_SMD:SOT-23-5_HandSoldering -> (none)
- R1, R10, R11, R12, R13, R14, R15, R16, R17, R18, R19, R2, R20, R21, R22, R23, R24, R25, R26, R27, R28, R3, R4, R5, R6, R7, R8, R9: footprint Resistors_SMD:R_0603_HandSoldering -> (none)
- SW1, SW10, SW2, SW9: footprint Buttons_Switches_THT:SW_PUSH_6mm -> (none)
- SW11, SW13, SW5, SW6: footprint mylib:dpad-h -> (none)
- SW12, SW14, SW3, SW4: footprint mylib:dpad-v -> (none)
- SW7, SW8: footprint Buttons_Switches_SMD:SW_SPST_TL3342 -> (none)
- U2: footprint Housings_SSOP:SOP-16_4.4x10.4mm_Pitch1.27mm -> (none)
- U3: footprint mylib:fpc-45pin-0.5mm-down -> (none)
- U4: footprint mylib:cm3354 -> (none)
- U5: footprint mylib:sc-70-5 -> (none)
Connections:
- wire segments 40 -> 39
Other:
- moved on the sheet: C1, C10, C11, C12, C2, C3, C4, C5, C6, C7, C8, C9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

Commit message: 20171208
Parts:
- SW1: value POWER -> Power
Changed lines of the file:
@@
 Sheet 1 1
 Title ""
-Date "7 dec 2017"
+Date "8 dec 2017"
 Rev ""
 Comp ""
@@
 P 11800 9100
 F 0 "SW1" H 11850 9200 50  0000 L CNN
-F 1 "POWER" H 11800 9040 50  0000 C CNN
+F 1 "Power" H 11800 9040 50  0000 C CNN
 F 2 "" H 11800 9300 50  0001 C CNN
 F 3 "" H 11800 9300 50  0001 C CNN
