File: q30/main.kicad_pcb (KiCad board)
At the start: 2 copper layers, 85.1 x 25.4 mm, 29 parts, among them J1 USB_B, SW1 UP, SW10 L, SW11 R, SW12 SELECT, SW13 START, SW14 BK1, SW15 BK2, SW16 BK3, SW17 BK4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

Commit message: 20171204
Parts:
- moved SW5 2.54 mm to (108.0, 144.8)
- moved SW1 2.54 mm to (162.6, 137.2)
- moved SW2 2.54 mm to (162.6, 152.4)
- moved SW3 2.54 mm to (170.2, 144.8)
- moved SW4 2.54 mm to (154.9, 144.8)
- moved SW6 2.54 mm to (115.6, 152.4)
- moved SW8 2.54 mm to (115.6, 137.2)
- moved SW9 2.54 mm to (123.2, 144.8)
Changed lines of the file:
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@@
   )
   (module mylib:dpad-v (layer B.Cu)
-    (at 165.1 137.16)
+    (at 162.56 137.16)
     (fp_text reference SW1 (at 0.07874 4.68584) (layer B.SilkS)
       (effects (font (size 1 1) (thickness 0.15)) (justify mirror))
@@
   )
   (module mylib:dpad-v (layer B.Cu)
-    (at 165.1 152.4)
+    (at 162.56 152.4)
     (fp_text reference SW2 (at 0.07874 4.68584) (layer B.SilkS)
       (effects (font (size 1 1) (thickness 0.15)) (justify mirror))
@@
   )
   (module mylib:dpad-h (layer B.Cu)
-    (at 172.72 144.78)
+    (at 170.18 144.78)
     (fp_text reference SW3 (at 0.12874 4.58584) (layer B.SilkS)
       (effects (font (size 1 1) (thickness 0.15)) (justify mirror))
@@
   )
   (module mylib:dpad-h (layer B.Cu)
-    (at 157.48 144.78)
+    (at 154.94 144.78)
     (fp_text reference SW4 (at 0.12874 4.58584) (layer B.SilkS)
       (effects (font (size 1 1) (thickness 0.15)) (justify mirror))
@@
   )
   (module mylib:dpad-h (layer B.Cu)
-    (at 105.41 144.78)
+    (at 107.95 144.78)
     (fp_text reference SW5 (at 0.12874 4.58584) (layer B.SilkS)
       (effects (font (size 1 1) (thickness 0.15)) (justify mirror))
@@
   )
   (module mylib:dpad-v (layer B.Cu)
-    (at 113.03 152.4)
+    (at 115.57 152.4)
     (fp_text reference SW6 (at 0.07874 4.68584) (layer B.SilkS)
       (effects (font (size 1 1) (thickness 0.15)) (justify mirror))
@@
   )
   (module mylib:dpad-v (layer B.Cu)
-    (at 113.03 137.16)
+    (at 115.57 137.16)
     (fp_text reference SW8 (at 0.07874 4.68584) (layer B.SilkS)
       (effects (font (size 1 1) (thickness 0.15)) (justify mirror))
@@
   )
   (module mylib:dpad-h (layer B.Cu)
-    (at 120.65 144.78)
+    (at 123.19 144.78)
     (fp_text reference SW9 (at 0.12874 4.58584) (layer B.SilkS)
       (effects (font (size 1 1) (thickness 0.15)) (justify mirror))
