File: q30/main.kicad_pcb (KiCad board)
At the start: 2 copper layers, 85.1 x 25.4 mm, 29 parts, among them J1 USB_B, SW1 UP, SW10 L, SW11 R, SW12 SELECT, SW13 START, SW14 BK1, SW15 BK2, SW16 BK3, SW17 BK4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

Commit message: 20171204
Parts:
- J1: footprint Connectors:USB_Mini-B -> mylib:miniusb-b
- U1: footprint Housings_DFN_QFN:QFN-48-1EP_7x7mm_Pitch0.5mm -> mylib:qfn-48-1ep_7x7mm_pitch0.5mm
- moved C6 0.32 mm to (153.6, 135.6), turned to 90 degrees
- moved C7 0.30 mm to (158.8, 135.6), turned to 90 degrees
Connections:
- U1 pad 1: (no net) -> Net-(U1-Pad1)
- U1 pad 2: (no net) -> Net-(U1-Pad2)
- U1 pad 28: (no net) -> Net-(U1-Pad28)
- U1 pad 29: (no net) -> Net-(U1-Pad29)
- U1 pad 3: (no net) -> Net-(U1-Pad3)
- U1 pad 30: (no net) -> Net-(U1-Pad30)
- U1 pad 31: (no net) -> Net-(U1-Pad31)
- U1 pad 34: (no net) -> Net-(U1-Pad34)
- U1 pad 37: (no net) -> Net-(U1-Pad37)
- U1 pad 38: (no net) -> Net-(U1-Pad38)
- U1 pad 39: (no net) -> Net-(U1-Pad39)
- U1 pad 4: (no net) -> Net-(U1-Pad4)
- U1 pad 40: (no net) -> Net-(U1-Pad40)
- U1 pad 41: (no net) -> Net-(U1-Pad41)
- U1 pad 42: (no net) -> Net-(U1-Pad42)
- U1 pad 43: (no net) -> Net-(U1-Pad43)
- U1 pad 45: (no net) -> Net-(U1-Pad45)
- U1 pad 46: (no net) -> Net-(U1-Pad46)
Routing:
- net GND: track 0.00 -> 82.1 mm
- net RST: track 0.00 -> 12.4 mm
- net Net-(C5-Pad2): track 0.00 -> 9.46 mm
- net +3V3: track 0.00 -> 7.46 mm
- net START: track 0.00 -> 6.50 mm
- net SELECT: track 0.00 -> 6.50 mm
- net R: track 0.00 -> 6.50 mm
- net L: track 0.00 -> 6.50 mm
- net BK4: track 0.00 -> 6.50 mm
- net BK3: track 0.00 -> 6.50 mm
- net BK2: track 0.00 -> 6.50 mm
- net BK1: track 0.00 -> 6.50 mm

Commit message: 20171205
Parts:
- moved U2 55.0 mm to (177.7, 144.8)
- moved J1 31.9 mm to (155.1, 153.0)
- moved R1 14.8 mm to (166.5, 156.5)
- moved C5 2.97 mm to (170.4, 156.5), turned to 0 degrees
- moved C2 1.73 mm to (158.4, 145.5), turned to 180 degrees
- moved C3 1.20 mm to (168.8, 149.5)
- moved C4 1.17 mm to (169.9, 141.1)
- moved SW7 0.76 mm to (174.0, 151.9)
- moved C1 0.28 mm to (163.6, 139.8)
Connections:
- U1 pad 10: UP -> RIGHT
- U1 pad 11: DOWN -> SELECT
- U1 pad 12: LEFT -> DOWN
- U1 pad 13: RIGHT -> Net-(U1-Pad13)
- U1 pad 18: L -> Net-(U1-Pad18)
- U1 pad 2: Net-(U1-Pad2) -> UP
- U1 pad 20: START -> Net-(U1-Pad20)
- U1 pad 21: SELECT -> Net-(U1-Pad21)
- U1 pad 22: BK1 -> START
- U1 pad 25: BK2 -> Net-(U1-Pad25)
- U1 pad 26: BK3 -> Net-(U1-Pad26)
- U1 pad 27: BK4 -> Net-(U1-Pad27)
- U1 pad 34: Net-(U1-Pad34) -> BK2
- U1 pad 37: Net-(U1-Pad37) -> LEFT
- U1 pad 38: Net-(U1-Pad38) -> BK4
- U1 pad 39: Net-(U1-Pad39) -> L
- U1 pad 40: Net-(U1-Pad40) -> BK1
- U1 pad 41: Net-(U1-Pad41) -> BK3
Routing:
- net GND: track 82.1 -> 239.7 mm, vias 0 -> 1
- net USB_DP: track 0.00 -> 31.6 mm, vias 0 -> 2
- net USB_DM: track 0.00 -> 30.4 mm
- net START: track 6.50 -> 36.4 mm
- net +5V: track 0.00 -> 28.1 mm
- net BK3: track 6.50 -> 28.5 mm, vias 0 -> 1
- net BK1: track 6.50 -> 26.5 mm
- net X2: track 0.00 -> 15.8 mm
- net SELECT: track 6.50 -> 16.8 mm
- net X1: track 0.00 -> 10.3 mm
- net L: track 6.50 -> 14.8 mm
- net RIGHT: track 0.00 -> 8.01 mm, vias 0 -> 1
- net Net-(C5-Pad2): track 9.46 -> 2.83 mm
- net R: track 6.50 -> 0.00 mm
- net BK4: track 6.50 -> 0.00 mm
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Other:
- board text added: "20171205"
- board text removed: "20171204"

Commit message: 20171207
Parts:
- C1, C2, C3, C4, C5, C6, C7: footprint Capacitors_SMD:C_0603_HandSoldering -> MyFT_C_0603
- J1: footprint mylib:miniusb-b -> MyFT_MiniUSB_B
- R1: footprint Resistors_SMD:R_0603_HandSoldering -> MyFT_R_0603
- SW1, SW2, SW6, SW8: footprint mylib:dpad-v -> MyFT_DPAD_TB; moved to F.Cu
- SW10, SW11, SW12, SW13, SW14, SW15, SW16, SW17, SW7: footprint Buttons_Switches_THT:SW_PUSH_6mm -> MyFT_SW_PUSH_6mm
- SW3, SW4, SW5, SW9: footprint mylib:dpad-h -> MyFT_DPAD_LR; moved to F.Cu
- U1: footprint mylib:qfn-48-1ep_7x7mm_pitch0.5mm -> MyFT_QFN-48-1EP_7x7mm_Pitch0.5mm
- U2: footprint TO_SOT_Packages_SMD:SOT-223 -> MyFT_SOT-223
- Y1: footprint Crystals:Crystal_SMD_5032-2pin_5.0x3.2mm_HandSoldering -> MyFT_Crystal_SMD_5032_2Pads
- moved SW8 284.8 mm to (375.9, 252.7)
- moved SW5 271.5 mm to (360.7, 243.8)
- moved SW6 263.0 mm to (358.1, 254.0)
- moved SW15 251.6 mm to (348.0, 260.4)
- moved SW4 248.0 mm to (382.3, 243.8)
- moved SW9 245.4 mm to (342.9, 254.0)
- moved SW11 234.6 mm to (309.9, 233.7)
- moved SW1 234.4 mm to (365.8, 254.0)
- moved SW17 233.9 mm to (332.7, 260.4)
- moved SW10 232.3 mm to (383.5, 233.7)
- moved U1 223.4 mm to (374.6, 222.2)
- moved Y1 222.1 mm to (354.3, 240.0)
- moved SW7 221.0 mm to (383.5, 222.2)
- moved SW12 220.9 mm to (351.8, 217.2)
- moved SW13 218.5 mm to (339.1, 217.2)
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Connections:
- net +3V3 renamed +3.3V
- C5 pad 2: Net-(C5-Pad2) -> GND
- SW7 pad 2: Net-(C5-Pad2) -> GND
- U1 pad 1: Net-(U1-Pad1) -> (no net)
- U1 pad 13: Net-(U1-Pad13) -> (no net)
- U1 pad 18: Net-(U1-Pad18) -> (no net)
- U1 pad 20: Net-(U1-Pad20) -> (no net)
- U1 pad 21: Net-(U1-Pad21) -> (no net)
- U1 pad 25: Net-(U1-Pad25) -> (no net)
- U1 pad 26: Net-(U1-Pad26) -> (no net)
- U1 pad 27: Net-(U1-Pad27) -> (no net)
- U1 pad 28: Net-(U1-Pad28) -> (no net)
- U1 pad 29: Net-(U1-Pad29) -> (no net)
- U1 pad 3: Net-(U1-Pad3) -> (no net)
- U1 pad 30: Net-(U1-Pad30) -> (no net)
- U1 pad 31: Net-(U1-Pad31) -> (no net)
- U1 pad 4: Net-(U1-Pad4) -> (no net)
- U1 pad 42: Net-(U1-Pad42) -> (no net)
- U1 pad 43: Net-(U1-Pad43) -> (no net)
- U1 pad 45: Net-(U1-Pad45) -> (no net)
- U1 pad 46: Net-(U1-Pad46) -> (no net)
Routing:
- net GND: track 239.7 -> 0.00 mm, vias 1 -> 0
- net START: track 36.4 -> 0.00 mm
- net USB_DP: track 31.6 -> 0.00 mm, vias 2 -> 0
- net USB_DM: track 30.4 -> 0.00 mm
- net BK3: track 28.5 -> 0.00 mm, vias 1 -> 0
- net +5V: track 28.1 -> 0.00 mm
- net BK1: track 26.5 -> 0.00 mm
- net SELECT: track 16.8 -> 0.00 mm
- net RST: track 16.3 -> 0.00 mm
- net X2: track 15.8 -> 0.00 mm
- net L: track 14.8 -> 0.00 mm
- net +3.3V: track 13.6 -> 0.00 mm
- net X1: track 10.3 -> 0.00 mm
- net RIGHT: track 8.01 -> 0.00 mm, vias 1 -> 0
- net UP: track 6.36 -> 0.00 mm, vias 1 -> 0
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Other:
- net class Default: clearance 0.2 -> 0.254; trace_width 0.25 -> 0.254; via_dia 0.6 -> 0.889; via_drill 0.4 -> 0.635
- rule trace_clearance: 0.2 -> 0.254
- rule trace_min: 0.2 -> 0.254
- rule via_min_drill: 0.3 -> 0.508
- rule via_min_size: 0.4 -> 0.889
- board text added: "USB Gamepad for Blackberry Passport"
- board text removed: "1.0"
- board text removed: "20171205"
- board text removed: "USB Gamdpad for Blackberry Passport"

Commit message: 20171219
Parts:
- added P1: CONN_4, SIL-4, F.Cu at (204.9, 124.3)
- J1: footprint MyFT_MiniUSB_B -> MyFT_USB_Mini_B_PIN_ONLY
- SW10, SW11, SW12, SW13, SW14, SW15, SW16, SW17, SW7: footprint MyFT_SW_PUSH_6mm -> MyFT_4.5x4.5_SMD
- U1: footprint MyFT_QFN-48-1EP_7x7mm_Pitch0.5mm -> MyFT_LQFP-48-1EP_7x7mm_Pitch0.5mm
- moved SW10 242.0 mm to (166.9, 125.8)
- moved U2 226.0 mm to (167.6, 143.6), turned to 180 degrees
- moved SW1 223.1 mm to (183.4, 125.5)
- moved SW4 221.0 mm to (191.0, 133.1)
- moved SW3 206.5 mm to (175.8, 133.1)
- moved SW2 203.0 mm to (183.4, 140.7)
- moved SW8 195.4 mm to (227.6, 125.5)
- moved SW17 192.9 mm to (174.5, 150.1)
- moved U1 188.6 mm to (205.0, 139.8), turned to 180 degrees
- moved C4 188.1 mm to (198.9, 142.4), turned to 270 degrees
- moved SW16 187.7 mm to (166.9, 150.1)
- moved Y1 185.0 mm to (205.1, 130.7)
- moved C7 181.0 mm to (207.0, 127.6), turned to 180 degrees
- moved C3 175.1 mm to (204.0, 133.7), turned to 180 degrees
- moved SW6 172.9 mm to (227.6, 140.7)
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Connections:
- U1 pad 10: RIGHT -> (no net)
- U1 pad 11: SELECT -> (no net)
- U1 pad 12: DOWN -> R
- U1 pad 13: (no net) -> L
- U1 pad 14: A -> (no net)
- U1 pad 15: B -> (no net)
- U1 pad 16: X -> (no net)
- U1 pad 17: Y -> (no net)
- U1 pad 19: R -> RIGHT
- U1 pad 2: UP -> X
- U1 pad 22: START -> (no net)
- U1 pad 26: (no net) -> DOWN
- U1 pad 27: (no net) -> UP
- U1 pad 28: (no net) -> LEFT
- U1 pad 29: (no net) -> BK3
- U1 pad 30: (no net) -> BK4
- U1 pad 31: (no net) -> SELECT
- U1 pad 34: BK2 -> SWDIO
- U1 pad 37: LEFT -> SWCLK
- U1 pad 38: BK4 -> START
- U1 pad 39: L -> B
- U1 pad 40: BK1 -> BK2
- U1 pad 41: BK3 -> BK1
- U1 pad 42: (no net) -> A
- U1 pad 46: (no net) -> Y
Other:
- board size 85.1 x 25.4 mm -> 84.8 x 30 mm
- net class Default: clearance 0.254 -> 0.18; trace_width 0.254 -> 0.18; via_dia 0.889 -> 0.6; via_drill 0.635 -> 0.4
- rule trace_clearance: 0.254 -> 0.18
- rule trace_min: 0.254 -> 0.18
- rule via_min_drill: 0.508 -> 0.4
- rule via_min_size: 0.889 -> 0.6
- board text removed: "USB Gamepad for Blackberry Passport"

Commit message: 20171219
Parts:
- moved C5 3.73 mm to (239.5, 143.3), turned to 270 degrees
- moved SW1 2.54 mm to (183.4, 128.0), turned to 180 degrees
- moved SW2 2.54 mm to (183.4, 143.3), turned to 180 degrees
- moved SW3 2.54 mm to (175.8, 135.6)
- moved SW4 2.54 mm to (191.0, 135.6)
- moved SW5 2.54 mm to (235.2, 135.6)
- moved SW6 2.54 mm to (227.6, 143.3)
- moved SW8 2.54 mm to (227.6, 128.0)
- moved SW9 2.54 mm to (220.0, 135.6)
- moved R1 1.49 mm to (242.5, 140.4)
- moved P1 0.85 mm to (205.3, 125.1)
- moved C2 0.76 mm to (208.2, 145.8)
- moved SW7 0.61 mm to (244.1, 143.9)
- moved U2 0.06 mm to (167.6, 143.7)
Connections:
- U1 pad 18: (no net) -> RIGHT
- U1 pad 19: RIGHT -> UP
- U1 pad 26: DOWN -> (no net)
- U1 pad 27: UP -> DOWN
- U1 pad 39: B -> BK2
- U1 pad 40: BK2 -> BK1
- U1 pad 41: BK1 -> B
Routing:
- net GND: track 0.00 -> 96.6 mm
- net R: track 0.00 -> 60.1 mm
- net L: track 0.00 -> 49.7 mm
- net +5V: track 0.00 -> 45.4 mm, vias 0 -> 2
- net BK1: track 0.00 -> 44.5 mm
- net BK3: track 0.00 -> 44.1 mm
- net LEFT: track 0.00 -> 38.7 mm
- net BK4: track 0.00 -> 36.9 mm
- net BK2: track 0.00 -> 36.3 mm
- net A: track 0.00 -> 28.9 mm
- net UP: track 0.00 -> 27.9 mm
- net X: track 0.00 -> 26.3 mm
- net DOWN: track 0.00 -> 22.3 mm
- net B: track 0.00 -> 19.6 mm
- net SELECT: track 0.00 -> 14.9 mm
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
Commit message: 20171220
Parts:
- added R2: 1.5K, MyFT_R_0603, F.Cu at (180.2, 149.0)
Routing:
- net GND: track 96.6 -> 353.5 mm, vias 0 -> 16
- net +3.3V: track 7.26 -> 161.6 mm, vias 0 -> 5
- net RST: track 9.04 -> 50.5 mm, vias 0 -> 2
- net USB_DP: track 13.2 -> 38.5 mm, vias 0 -> 2
- net SWCLK: track 0.00 -> 20.7 mm, vias 0 -> 1
- net SWDIO: track 0.00 -> 19.3 mm, vias 0 -> 1
- net X2: track 3.38 -> 14.0 mm, vias 0 -> 2
- net X1: track 3.38 -> 9.11 mm
- net START: track 13.2 -> 18.2 mm
- net +5V: track 45.4 -> 46.3 mm, vias 2 -> 3
- added copper zone on B.Cu, net GND
- added copper zone on F.Cu, net GND
