File: q30/main.sch (KiCad schematic (older format))
At the start: 29 parts, among them J1 USB_B, SW1 UP, SW10 L, SW11 R, SW12 SELECT, SW13 START, SW14 BK1, SW15 BK2, SW16 BK3, SW17 BK4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

Commit message: 20171204
Parts:
- J1: footprint Connectors:USB_Mini-B -> mylib:miniusb-b; symbol USB_B -> USB_B-RESCUE-main
- SW1, SW10, SW11, SW12, SW13, SW14, SW15, SW16, SW17, SW2, SW3, SW4, SW5, SW6, SW7, SW8, SW9: symbol SW_DPST_x2 -> SW_DPST_x2-RESCUE-main
- U1: footprint Housings_DFN_QFN:QFN-48-1EP_7x7mm_Pitch0.5mm -> mylib:qfn-48-1ep_7x7mm_pitch0.5mm
Changed lines of the file:
@@
 EESchema Schematic File Version 2
+LIBS:main-rescue
 LIBS:power
 LIBS:device
@@
 F 0 "U1" H 5650 3400 60  0000 C CNN
 F 1 "STM32F103_48PIN" H 5650 3300 60  0000 C CNN
-F 2 "Housings_DFN_QFN:QFN-48-1EP_7x7mm_Pitch0.5mm" H 5400 3800 60  0000 C CNN
+F 2 "mylib:qfn-48-1ep_7x7mm_pitch0.5mm" H 5400 3800 60  0000 C CNN
 F 3 "" H 5400 3800 60  0000 C CNN
 	1    5650 3350
@@
 $EndComp
 $Comp
-L SW_DPST_x2 SW7
+L SW_DPST_x2-RESCUE-main SW7
 U 1 1 5A24FB0F
 P 5050 5700
@@
 Connection ~ 5850 5350
 $Comp
-L USB_B J1
+L USB_B-RESCUE-main J1
 U 1 1 5A24FF7B
 P 7200 5300
 F 0 "J1" H 7000 5750 50  0000 L CNN
 F 1 "USB_B" H 7000 5650 50  0000 L CNN
-F 2 "Connectors:USB_Mini-B" H 7350 5250 50  0001 C CNN
+F 2 "mylib:miniusb-b" H 7350 5250 50  0001 C CNN
 F 3 "" H 7350 5250 50  0001 C CNN
 	1    7200 5300
@@
 $EndComp
 $Comp
-L SW_DPST_x2 SW1
+L SW_DPST_x2-RESCUE-main SW1
 U 1 1 5A250976
 P 3100 1600
@@
 $EndComp
 $Comp
-L SW_DPST_x2 SW2
+L SW_DPST_x2-RESCUE-main SW2
 U 1 1 5A2509BC
 P 3450 1600
@@
 $EndComp
 $Comp
-L SW_DPST_x2 SW3
+L SW_DPST_x2-RESCUE-main SW3
 U 1 1 5A250B09
 P 3800 1600
@@
 $EndComp
 $Comp
-L SW_DPST_x2 SW4
+L SW_DPST_x2-RESCUE-main SW4
 U 1 1 5A250B0F
 P 4150 1600
@@
 $EndComp
 $Comp
-L SW_DPST_x2 SW5
+L SW_DPST_x2-RESCUE-main SW5
 U 1 1 5A250BED
 P 4500 1600
@@
 $EndComp
 $Comp
-L SW_DPST_x2 SW6
+L SW_DPST_x2-RESCUE-main SW6
 U 1 1 5A250BF3
 P 4850 1600
@@
 $EndComp
 $Comp
-L SW_DPST_x2 SW8
+L SW_DPST_x2-RESCUE-main SW8
 U 1 1 5A250BF9
 P 5200 1600
@@
 $EndComp
 $Comp
-L SW_DPST_x2 SW9
+L SW_DPST_x2-RESCUE-main SW9
 U 1 1 5A250BFF
 P 5550 1600
@@
 $EndComp
 $Comp
-L SW_DPST_x2 SW10
+L SW_DPST_x2-RESCUE-main SW10
 U 1 1 5A2511F1
 P 5850 1600
@@
 $EndComp
 $Comp
-L SW_DPST_x2 SW11
+L SW_DPST_x2-RESCUE-main SW11
 U 1 1 5A2511F7
 P 6200 1600
@@
 $EndComp
 $Comp
-L SW_DPST_x2 SW12
+L SW_DPST_x2-RESCUE-main SW12
 U 1 1 5A2511FD
 P 6550 1600
@@
 $EndComp
 $Comp
-L SW_DPST_x2 SW13
+L SW_DPST_x2-RESCUE-main SW13
 U 1 1 5A251203
 P 6900 1600
@@
 $EndComp
 $Comp
-L SW_DPST_x2 SW14
+L SW_DPST_x2-RESCUE-main SW14
 U 1 1 5A25156F
 P 7200 1600
@@
 $EndComp
 $Comp
-L SW_DPST_x2 SW15
+L SW_DPST_x2-RESCUE-main SW15
 U 1 1 5A251575
 P 7550 1600
@@
 $EndComp
 $Comp
-L SW_DPST_x2 SW16
+L SW_DPST_x2-RESCUE-main SW16
 U 1 1 5A25157B
 P 7900 1600
@@
 $EndComp
 $Comp
-L SW_DPST_x2 SW17
+L SW_DPST_x2-RESCUE-main SW17
 U 1 1 5A251581
 P 8250 1600

Commit message: 20171205
Changed lines of the file:
@@
 Text GLabel 8250 1400 1    61   Input ~ 0
 BK4
+Text GLabel 4500 2950 0    60   Input ~ 0
+UP
+Text GLabel 4500 3950 0    60   Input ~ 0
+DOWN
+Text GLabel 6200 2300 1    60   Input ~ 0
+LEFT
 Text GLabel 4500 3750 0    60   Input ~ 0
-UP
-Text GLabel 4500 3850 0    60   Input ~ 0
-DOWN
-Text GLabel 4500 3950 0    60   Input ~ 0
-LEFT
-Text GLabel 5100 4500 3    60   Input ~ 0
 RIGHT
 Text GLabel 5200 4500 3    60   Input ~ 0
@@
 Text GLabel 5500 4500 3    60   Input ~ 0
 Y
-Text GLabel 5600 4500 3    60   Input ~ 0
+Text GLabel 6000 2300 1    60   Input ~ 0
 L
 Text GLabel 5700 4500 3    60   Input ~ 0
 R
-Text GLabel 5800 4500 3    60   Input ~ 0
+Text GLabel 6000 4500 3    60   Input ~ 0
 START
-Text GLabel 5900 4500 3    60   Input ~ 0
+Text GLabel 4500 3850 0    60   Input ~ 0
 SELECT
-Text GLabel 6000 4500 3    60   Input ~ 0
+Text GLabel 5900 2300 1    60   Input ~ 0
 BK1
-Text GLabel 6800 3950 2    60   Input ~ 0
+Text GLabel 6800 3050 2    60   Input ~ 0
 BK2
-Text GLabel 6800 3850 2    60   Input ~ 0
+Text GLabel 5800 2300 1    60   Input ~ 0
 BK3
-Text GLabel 6800 3750 2    60   Input ~ 0
+Text GLabel 6100 2300 1    60   Input ~ 0
 BK4
 NoConn ~ 6800 3650
@@
 NoConn ~ 6800 3450
 NoConn ~ 6800 3350
-NoConn ~ 6800 3050
-NoConn ~ 6200 2300
-NoConn ~ 6100 2300
-NoConn ~ 6000 2300
-NoConn ~ 5900 2300
-NoConn ~ 5800 2300
+NoConn ~ 6800 3750
+NoConn ~ 6800 3850
+NoConn ~ 5800 4500
+NoConn ~ 6800 3950
 NoConn ~ 5700 2300
 NoConn ~ 5600 2300
@@
 NoConn ~ 5300 2300
 NoConn ~ 4500 2850
-NoConn ~ 4500 2950
 NoConn ~ 4500 3050
 NoConn ~ 4500 3150
@@
 RST
 Connection ~ 5050 5500
+NoConn ~ 5100 4500
+NoConn ~ 5900 4500
+NoConn ~ 5600 4500
 $EndSCHEMATC

Commit message: 20171219
Parts:
- added P1: CONN_4, symbol CONN_4
- C1, C2, C3, C4, C5, C6, C7: footprint Capacitors_SMD:C_0603_HandSoldering -> (none)
- J1: footprint mylib:miniusb-b -> (none)
- R1: footprint Resistors_SMD:R_0603_HandSoldering -> (none)
- SW1, SW2, SW6, SW8: footprint mylib:dpad-v -> (none)
- SW10, SW11, SW12, SW13, SW14, SW15, SW16, SW17, SW7: footprint Buttons_Switches_THT:SW_PUSH_6mm -> (none)
- SW3, SW4, SW5, SW9: footprint mylib:dpad-h -> (none)
- U1: footprint mylib:qfn-48-1ep_7x7mm_pitch0.5mm -> (none)
- U2: footprint TO_SOT_Packages_SMD:SOT-223 -> (none)
- Y1: footprint Crystals:Crystal_SMD_5032-2pin_5.0x3.2mm_HandSoldering -> (none)
Connections:
- net labels added: SWCLK, SWDIO
- wire segments 6 -> 4
- no-connect marks 18 -> 16
Other:
- note added: "USB gamdpad for Blackberry Passport"
- note removed: "1.0"
- note removed: "20171204"
- note removed: "USB Gamdpad for Blackberry Passport"
- moved on the sheet: C1, C2, C3, C4, C5, R1, U2, Y1

Commit message: 20171219
Changed lines of the file:
@@
 Text GLabel 8250 1400 1    49   Input ~ 0
 BK4
+Text GLabel 5700 4500 3    49   Input ~ 0
+UP
 Text GLabel 6800 3750 2    49   Input ~ 0
-UP
-Text GLabel 6800 3850 2    49   Input ~ 0
 DOWN
 Text GLabel 6800 3650 2    49   Input ~ 0
 LEFT
-Text GLabel 5700 4500 3    49   Input ~ 0
+Text GLabel 5600 4500 3    49   Input ~ 0
 RIGHT
 Text GLabel 5700 2300 1    49   Input ~ 0
 A
-Text GLabel 6000 2300 1    49   Input ~ 0
+Text GLabel 5800 2300 1    49   Input ~ 0
 B
 Text GLabel 4500 2950 0    49   Input ~ 0
@@
 Text GLabel 6800 3350 2    49   Input ~ 0
 SELECT
-Text GLabel 5800 2300 1    49   Input ~ 0
+Text GLabel 5900 2300 1    49   Input ~ 0
 BK1
-Text GLabel 5900 2300 1    49   Input ~ 0
+Text GLabel 6000 2300 1    49   Input ~ 0
 BK2
 Text GLabel 6800 3550 2    49   Input ~ 0
@@
 Connection ~ 5050 5500
 NoConn ~ 5900 4500
-NoConn ~ 5600 4500
+NoConn ~ 6800 3850
 Connection ~ 6450 5300
 Connection ~ 5850 5300

Commit message: 20171220
Parts:
- added R2: 1.5K, ~, symbol R
Changed lines of the file:
@@
 Sheet 1 1
 Title ""
-Date "19 dec 2017"
+Date "20 dec 2017"
 Rev ""
 Comp ""
@@
 	-1   0    0    1
 $EndComp
+$Comp
+L R R2
+U 1 1 5A3A2831
+P 8150 5050
+F 0 "R2" V 8230 5050 40  0000 C CNN
+F 1 "1.5K" V 8157 5051 40  0000 C CNN
+F 2 "~" V 8080 5050 30  0000 C CNN
+F 3 "~" H 8150 5050 30  0000 C CNN
+	1    8150 5050
+	1    0    0    -1
+$EndComp
+$Comp
+L +5V #PWR031
+U 1 1 5A3A2858
+P 8150 4800
+F 0 "#PWR031" H 8150 4890 20  0001 C CNN
+F 1 "+5V" H 8150 4890 30  0000 C CNN
+F 2 "" H 8150 4800 60  0000 C CNN
+F 3 "" H 8150 4800 60  0000 C CNN
+	1    8150 4800
+	1    0    0    -1
+$EndComp
+Text GLabel 8150 5300 3    49   Input ~ 0
+USB_DP
 $EndSCHEMATC
