File: q20/main.kicad_pcb (KiCad board)
At the start: 2 copper layers, 65 x 35.1 mm, 29 parts, among them J1 USB_B, SW1 UP, SW10 L, SW11 R, SW12 SELECT, SW13 START, SW14 BK1, SW15 BK2, SW16 BK3, SW17 BK4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

Commit message: 20171219
Parts:
- added P1: CONN_4, SIL-4, F.Cu at (252.9, 161.7)
- U1: footprint MyFT_QFN-48-1EP_7x7mm_Pitch0.5mm -> MyFT_LQFP-48-1EP_7x7mm_Pitch0.5mm
- moved R1 6.44 mm to (258.6, 188.2), turned to 180 degrees
- moved C2 4.85 mm to (254.8, 184.2)
- moved C5 3.91 mm to (258.6, 186.6), turned to 0 degrees
- moved C1 3.87 mm to (258.2, 176.3)
- moved C4 3.78 mm to (246.1, 180.6)
- moved U1 3.62 mm to (252.2, 178.1), turned to 180 degrees
- moved C6 2.48 mm to (250.4, 165.9)
- moved Y1 2.48 mm to (252.3, 168.9)
- moved C7 2.48 mm to (254.3, 165.9)
- moved C3 2.36 mm to (251.2, 172.0)
Connections:
- U1 pad 34: (no net) -> SWDIO
- U1 pad 37: (no net) -> SWCLK
Routing:
- net GND: track 218.9 -> 0.00 mm, vias 6 -> 0
- net +3.3V: track 56.7 -> 0.00 mm, vias 2 -> 0
- net UP: track 51.5 -> 0.00 mm
- net BK1: track 48.7 -> 0.00 mm
- net R: track 48.1 -> 0.00 mm
- net BK3: track 44.4 -> 0.00 mm
- net LEFT: track 40.6 -> 0.00 mm
- net BK2: track 40.5 -> 0.00 mm
- net L: track 38.3 -> 0.00 mm
- net BK4: track 35.4 -> 0.00 mm
- net +5V: track 29.2 -> 0.00 mm, vias 2 -> 0
- net START: track 27.2 -> 0.00 mm
- net RST: track 25.5 -> 0.00 mm, vias 3 -> 0
- net DOWN: track 25.5 -> 0.00 mm
- net A: track 24.1 -> 0.00 mm
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
Commit message: 20171220
Parts:
- added R2: 1.5K, MyFT_R_0603, F.Cu at (229.8, 187.8)
- moved C2 0.77 mm to (255.5, 184.0)
- moved P1 0.51 mm to (252.7, 162.2)
- moved C3 0.15 mm to (251.1, 172.0)
Connections:
- U1 pad 25: (no net) -> DOWN
- U1 pad 26: DOWN -> (no net)
- U1 pad 39: B -> BK2
- U1 pad 40: BK2 -> BK1
- U1 pad 41: BK1 -> B
Routing:
- net GND: track 0.00 -> 313.7 mm, vias 0 -> 9
- net +3.3V: track 0.00 -> 107.8 mm, vias 0 -> 4
- net R: track 0.00 -> 52.4 mm
- net BK1: track 0.00 -> 43.3 mm
- net UP: track 0.00 -> 43.1 mm
- net L: track 0.00 -> 41.2 mm
- net BK3: track 0.00 -> 38.0 mm
- net LEFT: track 0.00 -> 36.6 mm
- net USB_DP: track 0.00 -> 35.6 mm, vias 0 -> 2
- net +5V: track 0.00 -> 35.2 mm, vias 0 -> 2
- net BK2: track 0.00 -> 35.0 mm
- net BK4: track 0.00 -> 31.0 mm
- net A: track 0.00 -> 29.5 mm
- net X: track 0.00 -> 24.2 mm
- net RST: track 0.00 -> 23.9 mm, vias 0 -> 3
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- added copper zone on B.Cu, net GND
- added copper zone on F.Cu, net GND
