File: q20/main.sch (KiCad schematic (older format))
At the start: 29 parts, among them J1 USB_B, SW1 UP, SW10 L, SW11 R, SW12 SELECT, SW13 START, SW14 BK1, SW15 BK2, SW16 BK3, SW17 BK4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

Commit message: 20171219
Parts:
- added P1: CONN_4, symbol CONN_4
Connections:
- net labels added: SWCLK, SWDIO
- no-connect marks 18 -> 16
Other:
- moved on the sheet: U2
Changed lines of the file:
@@
 Sheet 1 1
 Title ""
-Date "18 dec 2017"
+Date "19 dec 2017"
 Rev ""
 Comp ""
@@
 Text GLabel 6800 3450 2    49   Input ~ 0
 BK4
-NoConn ~ 6200 2300
 NoConn ~ 5600 2300
 NoConn ~ 6000 4500
@@
 L AMS1117-3.3 U2
 U 1 1 5A25AF73
-P 7225 4250
-F 0 "U2" H 7075 4550 60  0000 C CNN
-F 1 "AMS1117-3.3" H 7325 4450 60  0000 C CNN
-F 2 "" H 7275 4450 60  0000 C CNN
-F 3 "" H 7275 4450 60  0000 C CNN
-	1    7225 4250
+P 7975 4050
+F 0 "U2" H 7825 4350 60  0000 C CNN
+F 1 "AMS1117-3.3" H 8075 4250 60  0000 C CNN
+F 2 "" H 8025 4250 60  0000 C CNN
+F 3 "" H 8025 4250 60  0000 C CNN
+	1    7975 4050
 	1    0    0    -1
 $EndComp
@@
 L GND #PWR026
 U 1 1 5A25B006
-P 7125 4450
-F 0 "#PWR026" H 7125 4200 50  0001 C CNN
-F 1 "GND" V 7150 4300 50  0000 C CNN
-F 2 "" H 7125 4450 50  0001 C CNN
-F 3 "" H 7125 4450 50  0001 C CNN
-	1    7125 4450
+P 7875 4250
+F 0 "#PWR026" H 7875 4000 50  0001 C CNN
+F 1 "GND" V 7900 4100 50  0000 C CNN
+F 2 "" H 7875 4250 50  0001 C CNN
+F 3 "" H 7875 4250 50  0001 C CNN
+	1    7875 4250
 	1    0    0    -1
 $EndComp
@@
 L +3.3V #PWR027
 U 1 1 5A25B071
-P 7225 4450
-F 0 "#PWR027" H 7225 4300 50  0001 C CNN
-F 1 "+3.3V" V 7200 4675 50  0000 C CNN
-F 2 "" H 7225 4450 50  0001 C CNN
-F 3 "" H 7225 4450 50  0001 C CNN
-	1    7225 4450
+P 7975 4250
+F 0 "#PWR027" H 7975 4100 50  0001 C CNN
+F 1 "+3.3V" V 7950 4475 50  0000 C CNN
+F 2 "" H 7975 4250 50  0001 C CNN
+F 3 "" H 7975 4250 50  0001 C CNN
+	1    7975 4250
 	-1   0    0    1
 $EndComp
@@
 L +5V #PWR028
 U 1 1 5A25B0BF
-P 7325 4450
-F 0 "#PWR028" H 7325 4300 50  0001 C CNN
-F 1 "+5V" V 7300 4625 50  0000 C CNN
-F 2 "" H 7325 4450 50  0001 C CNN
-F 3 "" H 7325 4450 50  0001 C CNN
-	1    7325 4450
+P 8075 4250
+F 0 "#PWR028" H 8075 4100 50  0001 C CNN
+F 1 "+5V" V 8050 4425 50  0000 C CNN
+F 2 "" H 8075 4250 50  0001 C CNN
+F 3 "" H 8075 4250 50  0001 C CNN
+	1    8075 4250
 	-1   0    0    1
 $EndComp
@@
 RST
 Connection ~ 5050 5500
-NoConn ~ 6800 3050
 NoConn ~ 5900 4500
 NoConn ~ 5600 4500
 Connection ~ 6450 5300
 Connection ~ 5850 5300
+$Comp
+L CONN_4 P1
+U 1 1 5A38A19D
+P 7950 2700
+F 0 "P1" V 7900 2700 50  0000 C CNN
+F 1 "CONN_4" V 8000 2700 50  0000 C CNN
+F 2 "" H 7950 2700 60  0000 C CNN
+F 3 "" H 7950 2700 60  0000 C CNN
+	1    7950 2700
+	0    -1   -1   0
+$EndComp
+Text GLabel 6800 3050 2    49   Input ~ 0
+SWDIO
+Text GLabel 6200 2300 1    49   Input ~ 0
+SWCLK
+Text GLabel 7800 3050 3    49   Input ~ 0
+SWCLK
+Text GLabel 7900 3050 3    49   Input ~ 0
+SWDIO
+$Comp
+L GND #PWR029
+U 1 1 5A38A1AE
+P 8000 3050
+F 0 "#PWR029" H 8000 3050 30  0001 C CNN
+F 1 "GND" H 8000 2980 30  0001 C CNN
+F 2 "" H 8000 3050 60  0000 C CNN
+F 3 "" H 8000 3050 60  0000 C CNN
+	1    8000 3050
+	1    0    0    -1
+$EndComp
+$Comp
+L +3.3V #PWR030
+U 1 1 5A38A1BD
+P 8100 3050
+F 0 "#PWR030" H 8100 3010 30  0001 C CNN
+F 1 "+3.3V" H 8100 3160 30  0000 C CNN
+F 2 "" H 8100 3050 60  0000 C CNN
+F 3 "" H 8100 3050 60  0000 C CNN
+	1    8100 3050
+	-1   0    0    1
+$EndComp
 $EndSCHEMATC

Commit message: 20171220
Parts:
- added R2: 1.5K, ~, symbol R
Changed lines of the file:
@@
 Sheet 1 1
 Title ""
-Date "19 dec 2017"
+Date "20 dec 2017"
 Rev ""
 Comp ""
@@
 Text GLabel 6800 3750 2    49   Input ~ 0
 UP
-Text GLabel 6800 3850 2    49   Input ~ 0
+Text GLabel 6800 3950 2    49   Input ~ 0
 DOWN
 Text GLabel 6800 3650 2    49   Input ~ 0
@@
 Text GLabel 5700 2300 1    49   Input ~ 0
 A
-Text GLabel 6000 2300 1    49   Input ~ 0
+Text GLabel 5800 2300 1    49   Input ~ 0
 B
 Text GLabel 4500 2950 0    49   Input ~ 0
@@
 Text GLabel 6800 3350 2    49   Input ~ 0
 SELECT
-Text GLabel 5800 2300 1    49   Input ~ 0
+Text GLabel 5900 2300 1    49   Input ~ 0
 BK1
-Text GLabel 5900 2300 1    49   Input ~ 0
+Text GLabel 6000 2300 1    49   Input ~ 0
 BK2
 Text GLabel 6800 3550 2    49   Input ~ 0
@@
 NoConn ~ 4500 3750
 NoConn ~ 5800 4500
-NoConn ~ 6800 3950
+NoConn ~ 6800 3850
 NoConn ~ 5200 4500
 NoConn ~ 5300 4500
@@
 	-1   0    0    1
 $EndComp
+$Comp
+L R R2
+U 1 1 5A3A2461
+P 8050 5050
+F 0 "R2" V 8130 5050 40  0000 C CNN
+F 1 "1.5K" V 8057 5051 40  0000 C CNN
+F 2 "~" V 7980 5050 30  0000 C CNN
+F 3 "~" H 8050 5050 30  0000 C CNN
+	1    8050 5050
+	1    0    0    -1
+$EndComp
+$Comp
+L +5V #PWR031
+U 1 1 5A3A248D
+P 8050 4800
+F 0 "#PWR031" H 8050 4890 20  0001 C CNN
+F 1 "+5V" H 8050 4890 30  0000 C CNN
+F 2 "" H 8050 4800 60  0000 C CNN
+F 3 "" H 8050 4800 60  0000 C CNN
+	1    8050 4800
+	1    0    0    -1
+$EndComp
+Text GLabel 8050 5300 3    49   Input ~ 0
+USB_DP
 $EndSCHEMATC
